Commit message: super dinousaur

File: urdf/experiment.urdf (robot description, URDF)
Before this commit: robot body, 18 links, 17 joints
Links:
- added link head, mass 0.97559947; visual box size=0.125 0.08 0.0636
- added link neck, mass 0.97559947; visual box size=0.0357142857143 0.0142857142857 0.0151428571429
- added link tail, mass 0.97559947; visual mesh filename=package://simple_biped/cone.stl scale=0.005 0.005 0.005
- link body: geometry collision box size=0.25 0.1 0.106; visual box size=0.25 0.1 0.106
- link l_phalange: geometry collision box size=0.02 0.02 0.0745; visual box size=0.02 0.02 0.0745
- link r_phalange: geometry collision box size=0.02 0.02 0.0745; visual box size=0.02 0.02 0.0745
- link support: geometry collision box size=0.05 0.05 1.19; visual box size=0.05 0.05 1.19
Joints:
- added joint body_to_neck: type fixed, parent body, child neck, origin xyz=0.125 0 0.0353333333333 rpy=0 0 0
- added joint body_to_tail: type fixed, parent body, child tail, origin xyz=-0.125 0 0 rpy=0 0 0
- added joint neck_to_head: type fixed, parent neck, child head, origin xyz=0.0178571428571 0 0 rpy=0 0 0
- joint beam_to_support: origin xyz=0 0.503 -0.15 rpy=0 0 0 -> xyz=0 0.503 -0.595 rpy=0 0 0
- joint column_to_beam: axis (none) -> 0 0 1; type fixed -> continuous
- joint l_pelvis_joint: limit lower=-1.308996939 upper=0.785398163397 effort=10 velocity=5.6548668 -> lower=0 upper=0 effort=10 velocity=5.6548668; origin xyz=0 -0.075 0 rpy=0 0 0 -> xyz=-0.0416666666667 -0.05 0.0212 rpy=0 0 0
- joint l_phalange_joint: limit lower=-2.6179939 upper=2.6179939 effort=10 velocity=5.6548668 -> lower=-0.785398163397 upper=0 effort=10 velocity=5.6548668
- joint l_thigh_yaw_joint: limit lower=-2.6179939 upper=2.6179939 effort=10 velocity=5.6548668 -> lower=0 upper=0 effort=10 velocity=5.6548668
- joint r_pelvis_joint: limit lower=-1.308996939 upper=0.785398163397 effort=10 velocity=5.6548668 -> lower=0 upper=0 effort=10 velocity=5.6548668; origin xyz=0 0.075 0 rpy=0 0 0 -> xyz=-0.0416666666667 0.05 0.0212 rpy=0 0 0
- joint r_phalange_joint: limit lower=-2.6179939 upper=2.6179939 effort=10 velocity=5.6548668 -> lower=-0.785398163397 upper=0 effort=10 velocity=5.6548668
- joint r_thigh_yaw_joint: limit lower=-2.6179939 upper=2.6179939 effort=10 velocity=5.6548668 -> lower=0 upper=0 effort=10 velocity=5.6548668
- joint support_to_base_link: origin xyz=0 0 -0.15 rpy=0 0 0 -> xyz=0 0 -0.595 rpy=0 0 0

File: urdf/experiment.xacro (robot description, xacro)
@@ -5,7 +5,8 @@
   <xacro:include filename="$(find simple_biped)/urdf/gazebo.xacro" />
   <xacro:ros_control prefix="terop"/>
+  <xacro:property name="M_PI" value="3.1415926535897931" />
  <xacro:property name="body_height" value="0.106" />
- <xacro:property name="body_width" value="0.150" />
- <xacro:property name="body_large" value="0.300" />
+ <xacro:property name="body_width" value="0.100" />
+ <xacro:property name="body_large" value="0.250" />
   <xacro:property name="column_height" value="1.06" />
   <xacro:property name="cross_length" value="0.05" />
@@ -17,5 +18,62 @@
     <child link="column"/>
   </joint>
+  <link name="neck">
+    <inertial>
+      <origin xyz="-0.003053 -0.038651 -0.019268" />
+      <mass value="0.97559947"/>
+      <inertia ixx="3.1081800"  ixy="-0.25460189"  ixz="2.0318174" iyy="6.3787776" iyz="0.16417863" izz="5.3316425" />
+    </inertial>
+    <visual>
+      <origin xyz="0 0 0" rpy="0 0 0" />
+      <!--origin xyz="-0.0235 0 -0.03525" rpy="0 0 0" /-->
+      <geometry>
+        <box size="${body_large/7} ${body_width/7} ${body_height/7}" />
+      </geometry>
+    </visual>
+  </link>
+    <link name="head">
+    <inertial>
+      <origin xyz="-0.003053 -0.038651 -0.019268" />
+      <mass value="0.97559947"/>
+      <inertia ixx="3.1081800"  ixy="-0.25460189"  ixz="2.0318174" iyy="6.3787776" iyz="0.16417863" izz="5.3316425" />
+    </inertial>
+    <visual>
+      <origin xyz="${body_large*0.5/2} 0 0" rpy="0 0 0" />
+      <!--origin xyz="-0.0235 0 -0.03525" rpy="0 0 0" /-->
+      <geometry>
+        <box size="${body_large*0.5} ${body_width*0.8} ${body_height*0.6}" />
+      </geometry>
+    </visual>
+  </link>
+  <link name="tail">
+    <inertial>
+      <origin xyz="-0.003053 -0.038651 -0.019268" />
+      <mass value="0.97559947"/>
+      <inertia ixx="3.1081800"  ixy="-0.25460189"  ixz="2.0318174" iyy="6.3787776" iyz="0.16417863" izz="5.3316425" />
+    </inertial>
+    <visual>
+      <origin xyz="-0.250 0 0" rpy="0 ${-M_PI/2} 0" />
+      <!--origin xyz="-0.0235 0 -0.03525" rpy="0 0 0" /-->
+      <geometry>
+        <mesh filename="package://simple_biped/cone.stl" scale="0.005 0.005 0.005"/>
+      </geometry>
+    </visual>
+  </link>
   <link name="base_link"/>
+  <joint name="body_to_tail" type="fixed">
+    <parent link="body"/>
+    <child link="tail"/>
+    <origin xyz="${-body_large/2} 0 0" rpy="0 0 0" />
+  </joint>
+ <joint name="body_to_neck" type="fixed">
+    <parent link="body"/>
+    <child link="neck"/>
+    <origin xyz="${body_large/2} 0 ${body_height/3}" rpy="0 0 0" />
+  </joint>
+  <joint name="neck_to_head" type="fixed">
+    <parent link="neck"/>
+    <child link="head"/>
+    <origin xyz="${body_large/14} 0 0" rpy="0 0 0" />
+  </joint>
   <joint name="base_link_to_body" type="fixed">
     <parent link="base_link"/>

File: urdf/leg.xacro (robot description, xacro)
@@ -6,5 +6,4 @@
  <!--xacro:property name="body_width" value="0.109" /-->
  <!--xacro:property name="body_large" value="0.102" /-->
- <xacro:property name="M_PI" value="3.1415926535897931" />
 <xacro:property name="pelvis_height" value="0.028652" />
  <xacro:property name="pelvis_width" value="0.08175" />
@@ -149,5 +148,5 @@
     <parent link="${parent}"/>
     <child link="${side}_pelvis"/>
-    <origin xyz="0 ${reflect*body_width/2} 0" rpy="0 0 0" />
+    <origin xyz="${-body_large/6} ${reflect*body_width/2} ${body_height/5}" rpy="0 0 0" />
     <axis xyz="0 0 1" />
     <limit effort="10" velocity="5.6548668" lower="0" upper="0" />
