Commit message: fix little error, falta pensar los joints

File: urdf/structure.xacro (robot description, xacro)
@@ -6,5 +6,5 @@
   <xacro:property name="cross_length" value="0.025" />
   <xacro:property name="beam_height" value="10" />
-  <xacro:property name="support_height" value="0.25" />
+  <xacro:property name="support_height" value="0.80" />
   <xacro:macro name="structure" params="parent child body_height body_width body_large">
   <joint name="fixed" type="fixed">
@@ -34,7 +34,7 @@
     <parent link="beam"/>
     <child link="slider"/>
-    <origin xyz="0 0 0" rpy="0 0 0" />
-    <axis xyz="0 1 0" />
-    <limit effort="10" velocity="5.6548668" lower="0" upper="5" />
+    <origin xyz="0 0 0" rpy="0 0 ${90*M_PI/180}" />
+    <axis xyz="1 0 0" />
+    <limit effort="10" velocity="5.6548668" lower="3" upper="15" />
   </joint>
   <link name="column">
@@ -57,5 +57,22 @@
     </collision>
   </link>
-    <link name="slider"/>
+    <link name="slider">
+    <inertial>
+      <origin xyz="-0.003053 -0.038651 -0.019268" />
+      <mass value="0.97559947"/>
+      <inertia ixx="3.1081800"  ixy="-0.25460189"  ixz="2.0318174" iyy="6.3787776" iyz="0.16417863" izz="5.3316425" />
+    </inertial>
+    <visual>
+      <origin xyz="0 0 0" rpy="0 0 0" />
+      <geometry>
+        <box size="${cross_length} ${cross_length} ${cross_length}" />
+      </geometry>
+    </visual>
+    <collision>
+      <geometry>
+        <box size="${cross_length} ${cross_length} ${cross_length}" />
+      </geometry>
+    </collision>
+  </link>
     <link name="support">
     <inertial>

Commit message: testing

File: urdf/structure.xacro (robot description, xacro)
@@ -24,5 +24,5 @@
     <origin xyz="0 0 ${-1*(cross_length/2)}" rpy="0 0 0" />
     <axis xyz="0 1 0" />
-    <limit effort="3" velocity="1" lower="${-90*M_PI/180}" upper="${90*M_PI/180}" />
+    <limit effort="15" velocity="50" lower="${-90*M_PI/180}" upper="${90*M_PI/180}" />
   </joint>
   <joint name="support_to_base_link" type="fixed">
@@ -36,11 +36,11 @@
     <origin xyz="0 0 ${-1*cross_length}" rpy="0 0 ${90*M_PI/180}" />
     <axis xyz="1 0 0" />
-    <limit effort="3" velocity="3" lower="0.5" upper="20" />
+    <limit effort="3" velocity="2" lower="5" upper="20" />
   </joint>
   <link name="column">
     <inertial>
       <origin xyz="0 0 0" />
-      <mass value="0.8"/>
-      <xacro:cuboid_inertia_def x="${cross_length}" y="${cross_length}" z="${column_height}" mass="1000"/>
+      <mass value="1"/>
+      <xacro:cuboid_inertia_def x="${cross_length}" y="${cross_length}" z="${column_height}" mass="10"/>
     </inertial>
     <visual>
@@ -61,6 +61,6 @@
     <inertial>
       <origin xyz="0 0 0" />
-      <mass value="1"/>
-      <xacro:cuboid_inertia_def x="${cross_length}" y="${cross_length}" z="${cross_length}" mass="1"/>
+      <mass value="10"/>
+      <xacro:cuboid_inertia_def x="${cross_length}" y="${cross_length}" z="${cross_length}" mass="10"/>
     </inertial>
     <visual>
@@ -79,6 +79,6 @@
     <inertial>
       <origin xyz="0 0 ${-1*support_height/2}" />
-      <mass value="1"/>
-      <xacro:cuboid_inertia_def x="${cross_length}" y="${cross_length}" z="${support_height}" mass="1"/>
+      <mass value="10"/>
+      <xacro:cuboid_inertia_def x="${cross_length}" y="${cross_length}" z="${support_height}" mass="10"/>
     </inertial>
     <visual>
@@ -98,6 +98,6 @@
     <inertial>
       <origin xyz="0 ${beam_height/2} 0" />
-      <mass value="0.8"/>
-      <xacro:cuboid_inertia_def x="${cross_length}" y="${beam_height}" z="${cross_length}" mass="1000"/>
+      <mass value="2"/>
+      <xacro:cuboid_inertia_def x="${cross_length}" y="${beam_height}" z="${cross_length}" mass="10"/>
     </inertial>
     <visual>

Commit message: jesus lizard

File: urdf/structure.xacro (robot description, xacro)
@@ -8,5 +8,10 @@
   <xacro:property name="support_height" value="1.30" />
   <xacro:macro name="structure" params="parent child body_height body_width body_large">
+      <xacro:joint_pos_transmission joint="beam_to_slider"/>
     <gazebo reference="support_to_base_link">
+      <provideFeedback>true</provideFeedback>
+      <disableFixedJointLumping>true</disableFixedJointLumping>
+    </gazebo>
+      <gazebo reference="slider_to_support">
       <provideFeedback>true</provideFeedback>
       <disableFixedJointLumping>true</disableFixedJointLumping>
@@ -17,5 +22,5 @@
     <origin xyz="0 0 0" rpy="0 0 0" />
   </joint>
-  <joint name="column_to_beam" type="continuous">
+  <joint name="column_to_beam" type="fixed">
     <parent link="column"/>
     <child link="beam"/>
@@ -35,10 +40,10 @@
     <origin xyz="0 0 ${-support_height}" rpy="0 0 0" />
   </joint>
-  <joint name="beam_to_slider" type="fixed">
+  <joint name="beam_to_slider" type="prismatic">
     <parent link="beam"/>
     <child link="slider"/>
     <origin xyz="0 5 ${-1*cross_length}" rpy="0 0 0"/>
     <axis xyz="1 0 0" />
-    <!--limit effort="3" velocity="2" lower="5" upper="20" /-->
+    <limit effort="3" velocity="2" lower="5" upper="20" />
   </joint>
   <link name="column">

Commit message: testiiing

File: urdf/structure.xacro (robot description, xacro)
@@ -6,5 +6,5 @@
   <xacro:property name="cross_length" value="0.025" />
   <xacro:property name="beam_height" value="20" />
-  <xacro:property name="support_height" value="1.35" />
+  <xacro:property name="support_height" value="1.26" />
   <xacro:macro name="structure" params="parent child body_height body_width body_large">
     <xacro:joint_transmission joint="slider_to_support"/>

Commit message: casi caminando

File: urdf/structure.xacro (robot description, xacro)
@@ -5,5 +5,5 @@
   <xacro:property name="column_height" value="1.25" />
   <xacro:property name="cross_length" value="0.025" />
-  <xacro:property name="beam_height" value="20" />
+  <xacro:property name="beam_height" value="7" />
   <xacro:property name="support_height" value="1.30" />
   <xacro:macro name="structure" params="parent child body_height body_width body_large">
@@ -43,5 +43,5 @@
     <parent link="beam"/>
     <child link="slider"/>
-    <origin xyz="0 2 ${-1*cross_length}" rpy="0 0 0"/>
+    <origin xyz="0 5 ${-1*cross_length}" rpy="0 0 0"/>
     <axis xyz="1 0 0" />
     <!--limit effort="3" velocity="2" lower="5" upper="20" /-->

Commit message: test malo

File: urdf/structure.xacro (robot description, xacro)
@@ -106,5 +106,5 @@
     <link name="beam">
     <inertial>
-      <origin xyz="0 ${beam_height/2} 0" rpy="0 0 ${90*M_PI/180}"/>
+      <origin xyz="0 ${beam_height/2} 0" rpy="0 0 0"/>
       <mass value="8"/>
       <xacro:cuboid_inertia_def x="${cross_length}" y="${beam_height}" z="${cross_length}" mass="8"/>
