Commit message: biped malo

File: urdf/experiment.xacro (robot description, xacro)
@@ -11,5 +11,5 @@
   <xacro:property name="cross_length" value="0.05" />
   <xacro:property name="beam_height" value="1.006" />
-  <xacro:property name="support_height" value="0.300" />
+  <xacro:property name="support_height" value="1.190" />
   <link name="world"/>
   <joint name="fixed" type="fixed">
@@ -22,7 +22,8 @@
     <child link="body"/>
   </joint>
-  <joint name="column_to_beam" type="fixed">
+  <joint name="column_to_beam" type="continuous">
     <parent link="column"/>
     <child link="beam"/>
+    <axis xyz="0 0 1"/>
     <origin xyz="0 ${beam_height/2} ${column_height/2}" rpy="0 0 0" />
   </joint>

File: urdf/leg.xacro (robot description, xacro)
@@ -23,6 +23,6 @@
  <xacro:property name="ankle_large" value="0.045" />
    <xacro:property name="phalange_height" value="0.0745" />
- <xacro:property name="phalange_width" value="0.035" />
- <xacro:property name="phalange_large" value="0.045" />
+ <xacro:property name="phalange_width" value="0.020" />
+ <xacro:property name="phalange_large" value="0.020" />
   <xacro:macro name="leg" params="side parent reflect body_height body_width body_large">
       <!-- Transmissions -->
@@ -140,4 +140,5 @@
     </visual>
     <collision>
+      <origin xyz="0 0 ${-1*phalange_height/2}" rpy="0 0 0" />
       <geometry>
         <box size="${phalange_large} ${phalange_width} ${phalange_height}"/>
@@ -185,5 +186,5 @@
     <origin xyz="0 0 ${-1*ankle_height}" rpy="0 0 0" />
     <axis xyz="0 1 0" />
-    <limit effort="10" velocity="5.6548668" lower="-2.6179939" upper="2.6179939" />
+    <limit effort="10" velocity="5.6548668" lower="${-45*M_PI/180}" upper="0" />
   </joint>
 </xacro:macro>

Commit message: fixed the column and beam structure

File: urdf/experiment.xacro (robot description, xacro)
@@ -10,5 +10,5 @@
  <xacro:property name="body_large" value="0.250" />
   <xacro:property name="column_height" value="1.06" />
-  <xacro:property name="cross_length" value="0.05" />
+  <xacro:property name="cross_length" value="0.025" />
   <xacro:property name="beam_height" value="1.006" />
   <xacro:property name="support_height" value="1.190" />
@@ -17,4 +17,5 @@
     <parent link="world"/>
     <child link="column"/>
+    <origin xyz="0 0 0" rpy="0 0 0" />
   </joint>
   <link name="neck">
@@ -84,10 +85,10 @@
     <child link="beam"/>
     <axis xyz="0 0 1"/>
-    <origin xyz="0 ${beam_height/2} ${column_height/2}" rpy="0 0 0" />
+    <origin xyz="0 0 ${column_height/2}" rpy="0 0 0" />
   </joint>
     <joint name="beam_to_support" type="fixed">
     <parent link="beam"/>
     <child link="support"/>
-    <origin xyz="0 ${beam_height/2} ${-1*support_height/2}" rpy="0 0 0" />
+    <origin xyz="0 ${beam_height} ${-1*support_height/2}" rpy="0 0 0" />
   </joint>
   <joint name="support_to_base_link" type="fixed">
@@ -141,5 +142,5 @@
     <visual>
       <!--origin xyz="-0.0235 0 -0.03525" rpy="0 0 0" /-->
-      <origin xyz="0 0 0" rpy="0 0 0" />
+      <origin xyz="0 ${beam_height/2} 0" rpy="0 0 0" />
       <geometry>
         <box size="${cross_length} ${beam_height} ${cross_length} " />

Commit message: positions controllers for testing

File: urdf/experiment.xacro (robot description, xacro)
@@ -12,5 +12,5 @@
   <xacro:property name="cross_length" value="0.05" />
   <xacro:property name="beam_height" value="1.006" />
-  <xacro:property name="support_height" value="1.190" />
+  <xacro:property name="support_height" value="1.200" />
   <link name="world"/>
   <joint name="fixed" type="fixed">

File: urdf/leg.xacro (robot description, xacro)
@@ -26,10 +26,10 @@
   <xacro:macro name="leg" params="side parent reflect body_height body_width body_large">
       <!-- Transmissions -->
-    <xacro:joint_transmission joint="${side}_pelvis_joint"/>
-    <xacro:joint_transmission joint="${side}_thigh_yaw_joint"/>
-    <xacro:joint_transmission joint="${side}_thigh_pitch_joint"/>
-    <xacro:joint_transmission joint="${side}_tibia_joint"/>
-    <xacro:joint_transmission joint="${side}_ankle_joint"/>
-    <xacro:joint_transmission joint="${side}_phalange_joint"/>
+    <xacro:joint_pos_transmission joint="${side}_pelvis_joint"/>
+    <xacro:joint_pos_transmission joint="${side}_thigh_yaw_joint"/>
+    <xacro:joint_pos_transmission joint="${side}_thigh_pitch_joint"/>
+    <xacro:joint_pos_transmission joint="${side}_tibia_joint"/>
+    <xacro:joint_pos_transmission joint="${side}_ankle_joint"/>
+    <xacro:joint_pos_transmission joint="${side}_phalange_joint"/>
   <link name="${side}_pelvis" >
     <inertial>

Commit message: too much points

File: urdf/experiment.xacro (robot description, xacro)
@@ -12,5 +12,5 @@
   <xacro:property name="cross_length" value="0.025" />
   <xacro:property name="beam_height" value="1.006" />
-  <xacro:property name="support_height" value="1.200" />
+  <xacro:property name="support_height" value="1.000" />
   <link name="world"/>
   <joint name="fixed" type="fixed">

Commit message: is walking

File: urdf/experiment.xacro (robot description, xacro)
@@ -12,5 +12,5 @@
   <xacro:property name="cross_length" value="0.025" />
   <xacro:property name="beam_height" value="1.006" />
-  <xacro:property name="support_height" value="1.000" />
+  <xacro:property name="support_height" value="1.205" />
   <link name="world"/>
   <joint name="fixed" type="fixed">

File: urdf/leg.xacro (robot description, xacro)
@@ -26,10 +26,10 @@
   <xacro:macro name="leg" params="side parent reflect body_height body_width body_large">
       <!-- Transmissions -->
-    <xacro:joint_pos_transmission joint="${side}_pelvis_joint"/>
-    <xacro:joint_pos_transmission joint="${side}_thigh_yaw_joint"/>
-    <xacro:joint_pos_transmission joint="${side}_thigh_pitch_joint"/>
-    <xacro:joint_pos_transmission joint="${side}_tibia_joint"/>
-    <xacro:joint_pos_transmission joint="${side}_ankle_joint"/>
-    <xacro:joint_pos_transmission joint="${side}_phalange_joint"/>
+    <xacro:joint_transmission joint="${side}_pelvis_joint"/>
+    <xacro:joint_transmission joint="${side}_thigh_yaw_joint"/>
+    <xacro:joint_transmission joint="${side}_thigh_pitch_joint"/>
+    <xacro:joint_transmission joint="${side}_tibia_joint"/>
+    <xacro:joint_transmission joint="${side}_ankle_joint"/>
+    <xacro:joint_transmission joint="${side}_phalange_joint"/>
   <link name="${side}_pelvis" >
     <inertial>

Commit message: testing position controllers (doesnt work ok) and rearrange the experiment urdf

File: urdf/experiment.xacro (robot description, xacro)
@@ -9,148 +9,10 @@
  <xacro:property name="body_width" value="0.100" />
  <xacro:property name="body_large" value="0.250" />
-  <xacro:property name="column_height" value="1.06" />
-  <xacro:property name="cross_length" value="0.025" />
-  <xacro:property name="beam_height" value="1.006" />
-  <xacro:property name="support_height" value="1.205" />
   <link name="world"/>
-  <joint name="fixed" type="fixed">
-    <parent link="world"/>
-    <child link="column"/>
-    <origin xyz="0 0 0" rpy="0 0 0" />
-  </joint>
-  <link name="neck">
-    <inertial>
-      <origin xyz="-0.003053 -0.038651 -0.019268" />
-      <mass value="0.97559947"/>
-      <inertia ixx="3.1081800"  ixy="-0.25460189"  ixz="2.0318174" iyy="6.3787776" iyz="0.16417863" izz="5.3316425" />
-    </inertial>
-    <visual>
-      <origin xyz="0 0 0" rpy="0 0 0" />
-      <!--origin xyz="-0.0235 0 -0.03525" rpy="0 0 0" /-->
-      <geometry>
-        <box size="${body_large/7} ${body_width/7} ${body_height/7}" />
-      </geometry>
-    </visual>
-  </link>
-    <link name="head">
-    <inertial>
-      <origin xyz="-0.003053 -0.038651 -0.019268" />
-      <mass value="0.97559947"/>
-      <inertia ixx="3.1081800"  ixy="-0.25460189"  ixz="2.0318174" iyy="6.3787776" iyz="0.16417863" izz="5.3316425" />
-    </inertial>
-    <visual>
-      <origin xyz="${body_large*0.5/2} 0 0" rpy="0 0 0" />
-      <!--origin xyz="-0.0235 0 -0.03525" rpy="0 0 0" /-->
-      <geometry>
-        <box size="${body_large*0.5} ${body_width*0.8} ${body_height*0.6}" />
-      </geometry>
-    </visual>
-  </link>
-  <link name="tail">
-    <inertial>
-      <origin xyz="-0.003053 -0.038651 -0.019268" />
-      <mass value="0.97559947"/>
-      <inertia ixx="3.1081800"  ixy="-0.25460189"  ixz="2.0318174" iyy="6.3787776" iyz="0.16417863" izz="5.3316425" />
-    </inertial>
-    <visual>
-      <origin xyz="-0.250 0 0" rpy="0 ${-M_PI/2} 0" />
-      <!--origin xyz="-0.0235 0 -0.03525" rpy="0 0 0" /-->
-      <geometry>
-        <mesh filename="package://simple_biped/cone.stl" scale="0.005 0.005 0.005"/>
-      </geometry>
-    </visual>
-  </link>
   <link name="base_link"/>
-  <joint name="body_to_tail" type="fixed">
-    <parent link="body"/>
-    <child link="tail"/>
-    <origin xyz="${-body_large/2} 0 0" rpy="0 0 0" />
-  </joint>
- <joint name="body_to_neck" type="fixed">
-    <parent link="body"/>
-    <child link="neck"/>
-    <origin xyz="${body_large/2} 0 ${body_height/3}" rpy="0 0 0" />
-  </joint>
-  <joint name="neck_to_head" type="fixed">
-    <parent link="neck"/>
-    <child link="head"/>
-    <origin xyz="${body_large/14} 0 0" rpy="0 0 0" />
-  </joint>
   <joint name="base_link_to_body" type="fixed">
     <parent link="base_link"/>
     <child link="body"/>
   </joint>
-  <joint name="column_to_beam" type="continuous">
-    <parent link="column"/>
-    <child link="beam"/>
-    <axis xyz="0 0 1"/>
-    <origin xyz="0 0 ${column_height/2}" rpy="0 0 0" />
-  </joint>
-    <joint name="beam_to_support" type="fixed">
-    <parent link="beam"/>
-    <child link="support"/>
-    <origin xyz="0 ${beam_height} ${-1*support_height/2}" rpy="0 0 0" />
-  </joint>
-  <joint name="support_to_base_link" type="fixed">
-    <parent link="support"/>
-    <child link="base_link"/>
-    <origin xyz="0 0 ${-1*support_height/2}" rpy="0 0 0" />
-  </joint>
-  <link name="column">
-    <inertial>
-      <origin xyz="-0.003053 -0.038651 -0.019268" />
-      <mass value="0.97559947"/>
-      <inertia ixx="3.1081800"  ixy="-0.25460189"  ixz="2.0318174" iyy="6.3787776" iyz="0.16417863" izz="5.3316425" />
-    </inertial>
-    <visual>
-      <!--origin xyz="-0.0235 0 -0.03525" rpy="0 0 0" /-->
-      <origin xyz="0 0 0" rpy="0 0 0" />
-      <geometry>
-        <box size="${cross_length} ${cross_length} ${column_height}" />
-      </geometry>
-    </visual>
-    <collision>
-      <geometry>
-        <box size="${cross_length} ${cross_length} ${column_height}" />
-      </geometry>
-    </collision>
-  </link>
-    <link name="support">
-    <inertial>
-      <origin xyz="-0.003053 -0.038651 -0.019268" />
-      <mass value="0.97559947"/>
-      <inertia ixx="3.1081800"  ixy="-0.25460189"  ixz="2.0318174" iyy="6.3787776" iyz="0.16417863" izz="5.3316425" />
-    </inertial>
-    <visual>
-      <origin xyz="0 0 0" rpy="0 0 0" />
-      <geometry>
-        <box size="${cross_length} ${cross_length} ${support_height}" />
-      </geometry>
-    </visual>
-    <collision>
-      <geometry>
-        <box size="${cross_length} ${cross_length} ${support_height}" />
-      </geometry>
-    </collision>
-  </link>
-    <link name="beam">
-    <inertial>
-      <origin xyz="-0.003053 -0.038651 -0.019268" />
-      <mass value="0.97559947"/>
-      <inertia ixx="3.1081800"  ixy="-0.25460189"  ixz="2.0318174" iyy="6.3787776" iyz="0.16417863" izz="5.3316425" />
-    </inertial>
-    <visual>
-      <!--origin xyz="-0.0235 0 -0.03525" rpy="0 0 0" /-->
-      <origin xyz="0 ${beam_height/2} 0" rpy="0 0 0" />
-      <geometry>
-        <box size="${cross_length} ${beam_height} ${cross_length} " />
-      </geometry>
-    </visual>
-    <collision>
-      <geometry>
-        <box size="${cross_length} ${beam_height} ${cross_length} " />
-      </geometry>
-    </collision>
-  </link>
   <link name="body">
     <inertial>
@@ -172,7 +34,10 @@
     </collision>
   </link>
-    <!-- Arm -->
+  <xacro:include filename="$(find simple_biped)/urdf/structure.xacro"/>
   <xacro:include filename="$(find simple_biped)/urdf/leg.xacro" />
+  <xacro:include filename="$(find simple_biped)/urdf/details.xacro"/>
   <!-- Left Arm -->
+  <xacro:structure parent="world" child="base_link" body_height="${body_height}" body_width="${body_width}" body_large="${body_large}"/>
+  <xacro:details parent="body" body_height="${body_height}" body_width="${body_width}" body_large="${body_large}"/>
   <xacro:leg side="l" parent="body" reflect="-1" body_height="${body_height}" body_width="${body_width}" body_large="${body_large}"/>
   <!-- Right Arm -->

Commit message: ajuste de controladores

File: urdf/experiment.xacro (robot description, xacro)
@@ -40,6 +40,6 @@
   <xacro:structure parent="world" child="base_link" body_height="${body_height}" body_width="${body_width}" body_large="${body_large}"/>
   <xacro:details parent="body" body_height="${body_height}" body_width="${body_width}" body_large="${body_large}"/>
-  <xacro:leg side="l" parent="body" reflect="-1" body_height="${body_height}" body_width="${body_width}" body_large="${body_large}"/>
+  <xacro:leg side="l" parent="body" reflect="1" body_height="${body_height}" body_width="${body_width}" body_large="${body_large}"/>
   <!-- Right Arm -->
-   <xacro:leg side="r" parent="body" reflect="1" body_height="${body_height}" body_width="${body_width}" body_large="${body_large}"/>
+   <xacro:leg side="r" parent="body" reflect="-1" body_height="${body_height}" body_width="${body_width}" body_large="${body_large}"/>
 </robot>

File: urdf/leg.xacro (robot description, xacro)
@@ -139,6 +139,6 @@
     <inertial>
       <origin xyz="0 0 ${-1*phalange_height/2}" />
-      <mass value="0.2"/>
-      <xacro:cuboid_inertia_def x="${phalange_large}" y="${phalange_width}" z="${phalange_height}" mass="0.2"/>
+      <mass value="0.1"/>
+      <xacro:cuboid_inertia_def x="${phalange_large}" y="${phalange_width}" z="${phalange_height}" mass="0.1"/>
     </inertial>
     <visual>

File: urdf/structure.xacro (robot description, xacro)
@@ -6,5 +6,5 @@
   <xacro:property name="cross_length" value="0.025" />
   <xacro:property name="beam_height" value="20" />
-  <xacro:property name="support_height" value="1.00" />
+  <xacro:property name="support_height" value="1.35" />
   <xacro:macro name="structure" params="parent child body_height body_width body_large">
     <xacro:joint_transmission joint="slider_to_support"/>
@@ -43,5 +43,5 @@
     <parent link="beam"/>
     <child link="slider"/>
-    <origin xyz="0 5 ${-1*cross_length}" rpy="0 0 0"/>
+    <origin xyz="0 2 ${-1*cross_length}" rpy="0 0 0"/>
     <axis xyz="1 0 0" />
     <!--limit effort="3" velocity="2" lower="5" upper="20" /-->

Commit message: megh

File: urdf/experiment.xacro (robot description, xacro)
@@ -18,6 +18,6 @@
     <inertial>
       <origin xyz="0 0 0" />
-      <mass value="0.6"/>
-      <xacro:cuboid_inertia_def x="${body_large}" y="${body_width}" z="${body_height}" mass="0.6"/>
+      <mass value="0.8"/>
+      <xacro:cuboid_inertia_def x="${body_large}" y="${body_width}" z="${body_height}" mass="0.8"/>
     </inertial>
     <visual>

File: urdf/leg.xacro (robot description, xacro)
@@ -212,5 +212,5 @@
     <parent link="${side}_ankle"/>
     <child link="${side}_phalange"/>
-    <origin xyz="$0 0 ${-1*ankle_height}" rpy="0 0 0" />
+    <origin xyz="0 0 ${-1*ankle_height}" rpy="0 0 0" />
     <axis xyz="0 1 0" />
     <limit effort="8" velocity="6" lower="${-45*M_PI/180}" upper="0" />
