Commit message: limits of joint according to dinosaur

File: urdf/leg.xacro (robot description, xacro)
@@ -6,4 +6,5 @@
  <!--xacro:property name="body_width" value="0.109" /-->
  <!--xacro:property name="body_large" value="0.102" /-->
+ <xacro:property name="M_PI" value="3.1415926535897931" />
 <xacro:property name="pelvis_height" value="0.028652" />
  <xacro:property name="pelvis_width" value="0.08175" />
@@ -141,7 +142,7 @@
     <origin xyz="0 ${reflect*body_width/2} 0" rpy="0 0 0" />
     <axis xyz="0 0 1" />
-    <limit effort="10" velocity="5.6548668" lower="-2.6179939" upper="2.6179939" />
+    <limit effort="10" velocity="5.6548668" lower="${-75*M_PI/180}" upper="${45*M_PI/180}" />
   </joint>
-    <joint name="${side}_thigh_yaw_joint" type="revolute">
+  <joint name="${side}_thigh_yaw_joint" type="revolute">
     <parent link="${side}_pelvis"/>
     <child link="${side}_thigh_yaw"/>
@@ -155,5 +156,5 @@
     <origin xyz="0 0 0" rpy="0 0 0" />
     <axis xyz="0 1 0" />
-    <limit effort="10" velocity="5.6548668" lower="-2.6179939" upper="2.6179939" />
+    <limit effort="10" velocity="5.6548668" lower="${-75*M_PI/180}" upper="${45*M_PI/180}"  />
   </joint>
   <joint name="${side}_tibia_joint" type="revolute">
@@ -162,5 +163,5 @@
     <origin xyz="0 0 ${-1*thigh_height}" rpy="0 0 0" />
     <axis xyz="0 1 0" />
-    <limit effort="10" velocity="5.6548668" lower="-2.6179939" upper="2.6179939" />
+    <limit effort="10" velocity="5.6548668" lower="${0*M_PI/180}" upper="${150*M_PI/180}" />
   </joint>
   <joint name="${side}_ankle_joint" type="revolute">
@@ -169,5 +170,5 @@
     <origin xyz="0 0 ${-1*tibia_height}" rpy="0 0 0" />
     <axis xyz="0 1 0" />
-    <limit effort="10" velocity="5.6548668" lower="-2.6179939" upper="2.6179939" />
+    <limit effort="10" velocity="5.6548668" lower="${-90*M_PI/180}" upper="${0*M_PI/180}" />
   </joint>
   <joint name="${side}_phalange_joint" type="revolute">

File: urdf/terop_beta.urdf (robot description, URDF)
Before this commit: robot body, 14 links, 13 joints
Joints:
- joint l_ankle_joint: limit lower=-2.6179939 upper=2.6179939 effort=10 velocity=5.6548668 -> lower=-1.57079632679 upper=0.0 effort=10 velocity=5.6548668
- joint l_pelvis_joint: limit lower=-2.6179939 upper=2.6179939 effort=10 velocity=5.6548668 -> lower=-1.308996939 upper=0.785398163397 effort=10 velocity=5.6548668
- joint l_thigh_pitch_joint: limit lower=-2.6179939 upper=2.6179939 effort=10 velocity=5.6548668 -> lower=-1.308996939 upper=0.785398163397 effort=10 velocity=5.6548668
- joint l_tibia_joint: limit lower=-2.6179939 upper=2.6179939 effort=10 velocity=5.6548668 -> lower=0.0 upper=2.61799387799 effort=10 velocity=5.6548668
- joint r_ankle_joint: limit lower=-2.6179939 upper=2.6179939 effort=10 velocity=5.6548668 -> lower=-1.57079632679 upper=0.0 effort=10 velocity=5.6548668
- joint r_pelvis_joint: limit lower=-2.6179939 upper=2.6179939 effort=10 velocity=5.6548668 -> lower=-1.308996939 upper=0.785398163397 effort=10 velocity=5.6548668
- joint r_thigh_pitch_joint: limit lower=-2.6179939 upper=2.6179939 effort=10 velocity=5.6548668 -> lower=-1.308996939 upper=0.785398163397 effort=10 velocity=5.6548668
- joint r_tibia_joint: limit lower=-2.6179939 upper=2.6179939 effort=10 velocity=5.6548668 -> lower=0.0 upper=2.61799387799 effort=10 velocity=5.6548668

Commit message: final experiment on gazebo

File: urdf/leg.xacro (robot description, xacro)
@@ -27,4 +27,5 @@
   <xacro:macro name="leg" params="side parent reflect body_height body_width body_large">
       <!-- Transmissions -->
+    <xacro:joint_transmission joint="${side}_pelvis_joint"/>
     <xacro:joint_transmission joint="${side}_thigh_yaw_joint"/>
     <xacro:joint_transmission joint="${side}_thigh_pitch_joint"/>
@@ -120,4 +121,5 @@
     </visual>
     <collision>
+      <origin xyz="0 0 ${-1*ankle_height/2}" rpy="0 0 0" />
       <geometry>
         <box size="${ankle_large} ${ankle_width} ${ankle_height}"/>

Commit message: mal biped

File: urdf/leg.xacro (robot description, xacro)
@@ -151,5 +151,5 @@
     <origin xyz="0 ${reflect*body_width/2} 0" rpy="0 0 0" />
     <axis xyz="0 0 1" />
-    <limit effort="10" velocity="5.6548668" lower="${-75*M_PI/180}" upper="${45*M_PI/180}" />
+    <limit effort="10" velocity="5.6548668" lower="0" upper="0" />
   </joint>
   <joint name="${side}_thigh_yaw_joint" type="revolute">
@@ -158,5 +158,5 @@
     <origin xyz="0 ${reflect*pelvis_width/2} ${-1*pelvis_height}" rpy="0 0 0" />
     <axis xyz="0 0 1" />
-    <limit effort="10" velocity="5.6548668" lower="-2.6179939" upper="2.6179939" />
+    <limit effort="10" velocity="5.6548668" lower="0" upper="0" />
   </joint>
   <joint name="${side}_thigh_pitch_joint" type="revolute">

Commit message: finish him

File: urdf/leg.xacro (robot description, xacro)
@@ -150,5 +150,5 @@
     <origin xyz="${-body_large/6} ${reflect*body_width/2} ${body_height/5}" rpy="0 0 0" />
     <axis xyz="0 0 1" />
-    <limit effort="10" velocity="5.6548668" lower="0" upper="0" />
+    <limit effort="10" velocity="5.6548668" lower="0" upper="0.01" />
   </joint>
   <joint name="${side}_thigh_yaw_joint" type="revolute">
@@ -157,5 +157,5 @@
     <origin xyz="0 ${reflect*pelvis_width/2} ${-1*pelvis_height}" rpy="0 0 0" />
     <axis xyz="0 0 1" />
-    <limit effort="10" velocity="5.6548668" lower="0" upper="0" />
+    <limit effort="10" velocity="5.6548668" lower="0" upper="0.01" />
   </joint>
   <joint name="${side}_thigh_pitch_joint" type="revolute">

Commit message: biped vuela

File: urdf/leg.xacro (robot description, xacro)
@@ -42,6 +42,6 @@
     <inertial>
       <origin xyz="0 0 0" />
-      <mass value="0.1"/>
-      <xacro:cuboid_inertia_def x="${pelvis_large}" y="${pelvis_width}" z="${pelvis_height}" mass="100"/>
+      <mass value="0.3"/>
+      <xacro:cuboid_inertia_def x="${pelvis_large}" y="${pelvis_width}" z="${pelvis_height}" mass="0.3"/>
     </inertial>
     <visual>
@@ -61,6 +61,6 @@
     <inertial>
       <origin xyz="0 0 0" />
-      <mass value="0.01"/>
-      <xacro:cuboid_inertia_def x="${thigh_virtual_large}" y="${thigh_virtual_width}" z="${thigh_virtual_height}" mass="100"/>
+      <mass value="0.1"/>
+      <xacro:cuboid_inertia_def x="${thigh_virtual_large}" y="${thigh_virtual_width}" z="${thigh_virtual_height}" mass="0.6"/>
     </inertial>
     <visual>
@@ -79,6 +79,6 @@
     <inertial>
       <origin xyz="0 0 0" />
-      <mass value="0.2"/>
-      <xacro:cuboid_inertia_def x="${thigh_large}" y="${thigh_width}" z="${thigh_height}" mass="100"/>
+      <mass value="0.8"/>
+      <xacro:cuboid_inertia_def x="${thigh_large}" y="${thigh_width}" z="${thigh_height}" mass="0.8"/>
     </inertial>
     <visual>
@@ -98,6 +98,6 @@
     <inertial>
       <origin xyz="0 0 0" />
-      <mass value="0.15"/>
-      <xacro:cuboid_inertia_def x="${tibia_large}" y="${tibia_width}" z="${tibia_height}" mass="100"/>
+      <mass value="0.6"/>
+      <xacro:cuboid_inertia_def x="${tibia_large}" y="${tibia_width}" z="${tibia_height}" mass="0.6"/>
     </inertial>
     <visual>
@@ -117,6 +117,6 @@
     <inertial>
       <origin xyz="0 0 0" />
-      <mass value="0.1"/>
-      <xacro:cuboid_inertia_def x="${ankle_large}" y="${ankle_width}" z="${ankle_height}" mass="100"/>
+      <mass value="0.3"/>
+      <xacro:cuboid_inertia_def x="${ankle_large}" y="${ankle_width}" z="${ankle_height}" mass="0.3"/>
     </inertial>
     <visual>
@@ -136,6 +136,6 @@
     <inertial>
       <origin xyz="0 0 0" />
-      <mass value="0.05"/>
-      <xacro:cuboid_inertia_def x="${phalange_large}" y="${phalange_width}" z="${phalange_height}" mass="100"/>
+      <mass value="0.2"/>
+      <xacro:cuboid_inertia_def x="${phalange_large}" y="${phalange_width}" z="${phalange_height}" mass="0.2"/>
     </inertial>
     <visual>
@@ -157,5 +157,5 @@
     <origin xyz="${-body_large/6} ${reflect*body_width/2} ${body_height/5}" rpy="0 0 0" />
     <axis xyz="0 0 1" />
-    <limit effort="10" velocity="5.6548668" lower="0" upper="0.01" />
+    <limit effort="4" velocity="1" lower="0" upper="0.01" />
   </joint>
   <joint name="${side}_thigh_yaw_joint" type="revolute">
@@ -164,5 +164,5 @@
     <origin xyz="0 ${reflect*pelvis_width/2} ${-1*pelvis_height}" rpy="0 0 0" />
     <axis xyz="0 0 1" />
-    <limit effort="10" velocity="5.6548668" lower="0" upper="0.01" />
+    <limit effort="4" velocity="1" lower="0" upper="0.01" />
   </joint>
   <joint name="${side}_thigh_pitch_joint" type="revolute">
@@ -171,5 +171,5 @@
     <origin xyz="0 0 0" rpy="0 0 0" />
     <axis xyz="0 1 0" />
-    <limit effort="10" velocity="5.6548668" lower="${-75*M_PI/180}" upper="${45*M_PI/180}"  />
+    <limit effort="4" velocity="1" lower="${-75*M_PI/180}" upper="${45*M_PI/180}"  />
   </joint>
   <joint name="${side}_tibia_joint" type="revolute">
@@ -178,5 +178,5 @@
     <origin xyz="0 0 ${-1*thigh_height}" rpy="0 0 0" />
     <axis xyz="0 1 0" />
-    <limit effort="10" velocity="5.6548668" lower="${0*M_PI/180}" upper="${150*M_PI/180}" />
+    <limit effort="4" velocity="1" lower="${0*M_PI/180}" upper="${150*M_PI/180}" />
   </joint>
   <joint name="${side}_ankle_joint" type="revolute">
@@ -185,5 +185,5 @@
     <origin xyz="0 0 ${-1*tibia_height}" rpy="0 0 0" />
     <axis xyz="0 1 0" />
-    <limit effort="10" velocity="5.6548668" lower="${-90*M_PI/180}" upper="${0*M_PI/180}" />
+    <limit effort="4" velocity="1" lower="${-90*M_PI/180}" upper="${0*M_PI/180}" />
   </joint>
   <joint name="${side}_phalange_joint" type="revolute">
@@ -192,5 +192,5 @@
     <origin xyz="0 0 ${-1*ankle_height}" rpy="0 0 0" />
     <axis xyz="0 1 0" />
-    <limit effort="10" velocity="5.6548668" lower="${-45*M_PI/180}" upper="0" />
+    <limit effort="4" velocity="1" lower="${-45*M_PI/180}" upper="0" />
   </joint>
 </xacro:macro>

File: urdf/structure.xacro (robot description, xacro)
@@ -5,5 +5,5 @@
   <xacro:property name="column_height" value="1.25" />
   <xacro:property name="cross_length" value="0.025" />
-  <xacro:property name="beam_height" value="10" />
+  <xacro:property name="beam_height" value="20" />
   <xacro:property name="support_height" value="1.30" />
   <xacro:macro name="structure" params="parent child body_height body_width body_large">
@@ -24,5 +24,5 @@
     <origin xyz="0 0 ${-1*(cross_length/2)}" rpy="0 0 0" />
     <axis xyz="0 1 0" />
-    <limit effort="10" velocity="5.6548668" lower="${-90*M_PI/180}" upper="${90*M_PI/180}" />
+    <limit effort="3" velocity="1" lower="${-90*M_PI/180}" upper="${90*M_PI/180}" />
   </joint>
   <joint name="support_to_base_link" type="fixed">
@@ -36,5 +36,5 @@
     <origin xyz="0 0 ${-1*cross_length}" rpy="0 0 ${90*M_PI/180}" />
     <axis xyz="1 0 0" />
-    <limit effort="100" velocity="50.6548668" lower="3" upper="15" />
+    <limit effort="3" velocity="3" lower="0.5" upper="20" />
   </joint>
   <link name="column">
@@ -42,5 +42,5 @@
       <origin xyz="0 0 0" />
       <mass value="0.8"/>
-      <xacro:cuboid_inertia_def x="${cross_length}" y="${cross_length}" z="${column_height}" mass="100000"/>
+      <xacro:cuboid_inertia_def x="${cross_length}" y="${cross_length}" z="${column_height}" mass="1000"/>
     </inertial>
     <visual>
@@ -61,6 +61,6 @@
     <inertial>
       <origin xyz="0 0 0" />
-      <mass value="0.1"/>
-      <xacro:cuboid_inertia_def x="${cross_length}" y="${cross_length}" z="${cross_length}" mass="100000"/>
+      <mass value="1"/>
+      <xacro:cuboid_inertia_def x="${cross_length}" y="${cross_length}" z="${cross_length}" mass="1"/>
     </inertial>
     <visual>
@@ -79,6 +79,6 @@
     <inertial>
       <origin xyz="0 0 ${-1*support_height/2}" />
-      <mass value="0.8"/>
-      <xacro:cuboid_inertia_def x="${cross_length}" y="${cross_length}" z="${support_height}" mass="100"/>
+      <mass value="1"/>
+      <xacro:cuboid_inertia_def x="${cross_length}" y="${cross_length}" z="${support_height}" mass="1"/>
     </inertial>
     <visual>
@@ -99,5 +99,5 @@
       <origin xyz="0 ${beam_height/2} 0" />
       <mass value="0.8"/>
-      <xacro:cuboid_inertia_def x="${cross_length}" y="${beam_height}" z="${cross_length}" mass="100000"/>
+      <xacro:cuboid_inertia_def x="${cross_length}" y="${beam_height}" z="${cross_length}" mass="1000"/>
     </inertial>
     <visual>

Commit message: testing

File: urdf/leg.xacro (robot description, xacro)
@@ -24,4 +24,9 @@
  <xacro:property name="phalange_width" value="0.020" />
  <xacro:property name="phalange_large" value="0.020" />
+   <!-- Friction model from "Characterization and modeling of a Dynamixel servo" by Arno Mensin (model AX12, better than nothing) -->
+  <!-- Damping N.m.s/rad -->
+  <xacro:property name="dxl_damping" value="0.15" />
+  <!-- Friccion N.m -->
+  <xacro:property name="dxl_friction" value="0.3" />
   <xacro:macro name="cuboid_inertia_def" params="x y z mass">
     <inertia
@@ -152,17 +157,19 @@
     </collision>
   </link>
-  <joint name="${side}_pelvis_joint" type="revolute">
+  <joint name="${side}_pelvis_joint" type="fixed">
     <parent link="${parent}"/>
     <child link="${side}_pelvis"/>
     <origin xyz="${-body_large/6} ${reflect*body_width/2} ${body_height/5}" rpy="0 0 0" />
     <axis xyz="0 0 1" />
-    <limit effort="4" velocity="1" lower="0" upper="0.01" />
-  </joint>
-  <joint name="${side}_thigh_yaw_joint" type="revolute">
+    <!--limit effort="1" velocity="4" lower="0" upper="0.01" /-->
+    <!--dynamics damping="${dxl_damping}" friction="${dxl_friction}" /-->
+  </joint>
+  <joint name="${side}_thigh_yaw_joint" type="fixed">
     <parent link="${side}_pelvis"/>
     <child link="${side}_thigh_yaw"/>
     <origin xyz="0 ${reflect*pelvis_width/2} ${-1*pelvis_height}" rpy="0 0 0" />
     <axis xyz="0 0 1" />
-    <limit effort="4" velocity="1" lower="0" upper="0.01" />
+    <!--limit effort="1" velocity="4" lower="0" upper="0.01" /-->
+    <!--dynamics damping="${dxl_damping}" friction="${dxl_friction}" /-->
   </joint>
   <joint name="${side}_thigh_pitch_joint" type="revolute">
@@ -171,5 +178,6 @@
     <origin xyz="0 0 0" rpy="0 0 0" />
     <axis xyz="0 1 0" />
-    <limit effort="4" velocity="1" lower="${-75*M_PI/180}" upper="${45*M_PI/180}"  />
+    <limit effort="1" velocity="4" lower="${-75*M_PI/180}" upper="${45*M_PI/180}"  />
+    <!--dynamics damping="${dxl_damping}" friction="${dxl_friction}" /-->
   </joint>
   <joint name="${side}_tibia_joint" type="revolute">
@@ -178,5 +186,6 @@
     <origin xyz="0 0 ${-1*thigh_height}" rpy="0 0 0" />
     <axis xyz="0 1 0" />
-    <limit effort="4" velocity="1" lower="${0*M_PI/180}" upper="${150*M_PI/180}" />
+    <limit effort="1" velocity="4" lower="${0*M_PI/180}" upper="${150*M_PI/180}" />
+    <!--dynamics damping="${dxl_damping}" friction="${dxl_friction}" /-->
   </joint>
   <joint name="${side}_ankle_joint" type="revolute">
@@ -185,5 +194,6 @@
     <origin xyz="0 0 ${-1*tibia_height}" rpy="0 0 0" />
     <axis xyz="0 1 0" />
-    <limit effort="4" velocity="1" lower="${-90*M_PI/180}" upper="${0*M_PI/180}" />
+    <limit effort="1" velocity="4" lower="${-90*M_PI/180}" upper="${0*M_PI/180}" />
+    <!--dynamics damping="${dxl_damping}" friction="${dxl_friction}" /-->
   </joint>
   <joint name="${side}_phalange_joint" type="revolute">
@@ -192,5 +202,6 @@
     <origin xyz="0 0 ${-1*ankle_height}" rpy="0 0 0" />
     <axis xyz="0 1 0" />
-    <limit effort="4" velocity="1" lower="${-45*M_PI/180}" upper="0" />
+    <limit effort="1" velocity="4" lower="${-45*M_PI/180}" upper="0" />
+    <!--dynamics damping="${dxl_damping}" friction="${dxl_friction}" /-->
   </joint>
 </xacro:macro>

File: urdf/structure.xacro (robot description, xacro)
@@ -31,16 +31,16 @@
     <origin xyz="0 0 ${-support_height}" rpy="0 0 0" />
   </joint>
-  <joint name="beam_to_slider" type="prismatic">
+  <joint name="beam_to_slider" type="fixed">
     <parent link="beam"/>
     <child link="slider"/>
-    <origin xyz="0 0 ${-1*cross_length}" rpy="0 0 ${90*M_PI/180}" />
+    <origin xyz="0 0 ${-1*cross_length}" rpy="0 0 ${90*M_PI/180}"/>
     <axis xyz="1 0 0" />
-    <limit effort="3" velocity="2" lower="5" upper="20" />
+    <!--limit effort="3" velocity="2" lower="5" upper="20" /-->
   </joint>
   <link name="column">
     <inertial>
       <origin xyz="0 0 0" />
-      <mass value="1"/>
-      <xacro:cuboid_inertia_def x="${cross_length}" y="${cross_length}" z="${column_height}" mass="10"/>
+      <mass value="3"/>
+      <xacro:cuboid_inertia_def x="${cross_length}" y="${cross_length}" z="${column_height}" mass="3"/>
     </inertial>
     <visual>
@@ -61,6 +61,6 @@
     <inertial>
       <origin xyz="0 0 0" />
-      <mass value="10"/>
-      <xacro:cuboid_inertia_def x="${cross_length}" y="${cross_length}" z="${cross_length}" mass="10"/>
+      <mass value="0.1"/>
+      <xacro:cuboid_inertia_def x="${cross_length}" y="${cross_length}" z="${cross_length}" mass="0.1"/>
     </inertial>
     <visual>
@@ -78,7 +78,7 @@
     <link name="support">
     <inertial>
-      <origin xyz="0 0 ${-1*support_height/2}" />
-      <mass value="10"/>
-      <xacro:cuboid_inertia_def x="${cross_length}" y="${cross_length}" z="${support_height}" mass="10"/>
+      <origin xyz="0 0 0" />
+      <mass value="0.4"/>
+      <xacro:cuboid_inertia_def x="${cross_length}" y="${cross_length}" z="${support_height}" mass="0.4"/>
     </inertial>
     <visual>
@@ -98,6 +98,6 @@
     <inertial>
       <origin xyz="0 ${beam_height/2} 0" />
-      <mass value="2"/>
-      <xacro:cuboid_inertia_def x="${cross_length}" y="${beam_height}" z="${cross_length}" mass="10"/>
+      <mass value="8"/>
+      <xacro:cuboid_inertia_def x="${cross_length}" y="${beam_height}" z="${cross_length}" mass="8"/>
     </inertial>
     <visual>

Commit message: caminan2

File: urdf/leg.xacro (robot description, xacro)
@@ -38,6 +38,4 @@
   <xacro:macro name="leg" params="side parent reflect body_height body_width body_large">
       <!-- Transmissions -->
-    <xacro:joint_transmission joint="${side}_pelvis_joint"/>
-    <xacro:joint_transmission joint="${side}_thigh_yaw_joint"/>
     <xacro:joint_transmission joint="${side}_thigh_pitch_joint"/>
     <xacro:joint_transmission joint="${side}_tibia_joint"/>
@@ -162,5 +160,5 @@
     <origin xyz="${-body_large/6} ${reflect*body_width/2} ${body_height/5}" rpy="0 0 0" />
     <axis xyz="0 0 1" />
-    <!--limit effort="1" velocity="4" lower="0" upper="0.01" /-->
+    <!--limit effort="4" velocity="4" lower="0" upper="0.01" /-->
     <!--dynamics damping="${dxl_damping}" friction="${dxl_friction}" /-->
   </joint>
@@ -170,5 +168,5 @@
     <origin xyz="0 ${reflect*pelvis_width/2} ${-1*pelvis_height}" rpy="0 0 0" />
     <axis xyz="0 0 1" />
-    <!--limit effort="1" velocity="4" lower="0" upper="0.01" /-->
+    <!--limit effort="4" velocity="4" lower="0" upper="0.01" /-->
     <!--dynamics damping="${dxl_damping}" friction="${dxl_friction}" /-->
   </joint>
@@ -178,5 +176,5 @@
     <origin xyz="0 0 0" rpy="0 0 0" />
     <axis xyz="0 1 0" />
-    <limit effort="1" velocity="4" lower="${-75*M_PI/180}" upper="${45*M_PI/180}"  />
+    <limit effort="4" velocity="4" lower="${-75*M_PI/180}" upper="${45*M_PI/180}"  />
     <!--dynamics damping="${dxl_damping}" friction="${dxl_friction}" /-->
   </joint>
@@ -186,5 +184,5 @@
     <origin xyz="0 0 ${-1*thigh_height}" rpy="0 0 0" />
     <axis xyz="0 1 0" />
-    <limit effort="1" velocity="4" lower="${0*M_PI/180}" upper="${150*M_PI/180}" />
+    <limit effort="4" velocity="4" lower="${0*M_PI/180}" upper="${150*M_PI/180}" />
     <!--dynamics damping="${dxl_damping}" friction="${dxl_friction}" /-->
   </joint>
@@ -194,5 +192,5 @@
     <origin xyz="0 0 ${-1*tibia_height}" rpy="0 0 0" />
     <axis xyz="0 1 0" />
-    <limit effort="1" velocity="4" lower="${-90*M_PI/180}" upper="${0*M_PI/180}" />
+    <limit effort="4" velocity="4" lower="${-90*M_PI/180}" upper="${0*M_PI/180}" />
     <!--dynamics damping="${dxl_damping}" friction="${dxl_friction}" /-->
   </joint>
@@ -202,5 +200,5 @@
     <origin xyz="0 0 ${-1*ankle_height}" rpy="0 0 0" />
     <axis xyz="0 1 0" />
-    <limit effort="1" velocity="4" lower="${-45*M_PI/180}" upper="0" />
+    <limit effort="4" velocity="4" lower="${-45*M_PI/180}" upper="0" />
     <!--dynamics damping="${dxl_damping}" friction="${dxl_friction}" /-->
   </joint>

File: urdf/structure.xacro (robot description, xacro)
@@ -13,5 +13,5 @@
     <origin xyz="0 0 0" rpy="0 0 0" />
   </joint>
-  <joint name="column_to_beam" type="fixed">
+  <joint name="column_to_beam" type="continuous">
     <parent link="column"/>
     <child link="beam"/>
@@ -19,10 +19,10 @@
     <origin xyz="0 0 ${column_height/2}" rpy="0 0 0" />
   </joint>
-    <joint name="slider_to_support" type="revolute">
+    <joint name="slider_to_support" type="fixed">
     <parent link="slider"/>
     <child link="support"/>
     <origin xyz="0 0 ${-1*(cross_length/2)}" rpy="0 0 0" />
     <axis xyz="0 1 0" />
-    <limit effort="15" velocity="50" lower="${-90*M_PI/180}" upper="${90*M_PI/180}" />
+    <!--limit effort="15" velocity="50" lower="${-90*M_PI/180}" upper="${90*M_PI/180}" /-->
   </joint>
   <joint name="support_to_base_link" type="fixed">
@@ -34,5 +34,5 @@
     <parent link="beam"/>
     <child link="slider"/>
-    <origin xyz="0 0 ${-1*cross_length}" rpy="0 0 ${90*M_PI/180}"/>
+    <origin xyz="0 1 ${-1*cross_length}" rpy="0 0 0"/>
     <axis xyz="1 0 0" />
     <!--limit effort="3" velocity="2" lower="5" upper="20" /-->

Commit message: caminan12 pro

File: urdf/leg.xacro (robot description, xacro)
@@ -139,6 +139,6 @@
     <inertial>
       <origin xyz="0 0 0" />
-      <mass value="0.2"/>
-      <xacro:cuboid_inertia_def x="${phalange_large}" y="${phalange_width}" z="${phalange_height}" mass="0.2"/>
+      <mass value="0.1"/>
+      <xacro:cuboid_inertia_def x="${phalange_large}" y="${phalange_width}" z="${phalange_height}" mass="0.1"/>
     </inertial>
     <visual>
@@ -176,5 +176,5 @@
     <origin xyz="0 0 0" rpy="0 0 0" />
     <axis xyz="0 1 0" />
-    <limit effort="4" velocity="4" lower="${-75*M_PI/180}" upper="${45*M_PI/180}"  />
+    <limit effort="8" velocity="6" lower="${-75*M_PI/180}" upper="${45*M_PI/180}"  />
     <!--dynamics damping="${dxl_damping}" friction="${dxl_friction}" /-->
   </joint>

File: urdf/structure.xacro (robot description, xacro)
@@ -34,5 +34,5 @@
     <parent link="beam"/>
     <child link="slider"/>
-    <origin xyz="0 1 ${-1*cross_length}" rpy="0 0 0"/>
+    <origin xyz="0 5 ${-1*cross_length}" rpy="0 0 0"/>
     <axis xyz="1 0 0" />
     <!--limit effort="3" velocity="2" lower="5" upper="20" /-->

Commit message: testing (no camina)

File: urdf/leg.xacro (robot description, xacro)
@@ -139,6 +139,6 @@
     <inertial>
       <origin xyz="0 0 ${-1*phalange_height/2}" />
-      <mass value="0.1"/>
-      <xacro:cuboid_inertia_def x="${phalange_large}" y="${phalange_width}" z="${phalange_height}" mass="0.1"/>
+      <mass value="0.2"/>
+      <xacro:cuboid_inertia_def x="${phalange_large}" y="${phalange_width}" z="${phalange_height}" mass="0.2"/>
     </inertial>
     <visual>
