Commit message: no explotando no caminando

File: urdf/leg.xacro (robot description, xacro)
@@ -184,5 +184,5 @@
     <origin xyz="0 0 ${-1*thigh_height}" rpy="0 0 0" />
     <axis xyz="0 1 0" />
-    <limit effort="4" velocity="4" lower="${0*M_PI/180}" upper="${150*M_PI/180}" />
+    <limit effort="8" velocity="6" lower="${0*M_PI/180}" upper="${150*M_PI/180}" />
     <!--dynamics damping="${dxl_damping}" friction="${dxl_friction}" /-->
   </joint>
@@ -192,5 +192,5 @@
     <origin xyz="0 0 ${-1*tibia_height}" rpy="0 0 0" />
     <axis xyz="0 1 0" />
-    <limit effort="4" velocity="4" lower="${-90*M_PI/180}" upper="${0*M_PI/180}" />
+    <limit effort="8" velocity="6" lower="${-90*M_PI/180}" upper="${0*M_PI/180}" />
     <!--dynamics damping="${dxl_damping}" friction="${dxl_friction}" /-->
   </joint>

File: urdf/structure.xacro (robot description, xacro)
@@ -6,7 +6,7 @@
   <xacro:property name="cross_length" value="0.025" />
   <xacro:property name="beam_height" value="20" />
-  <xacro:property name="support_height" value="1.30" />
+  <xacro:property name="support_height" value="1.00" />
   <xacro:macro name="structure" params="parent child body_height body_width body_large">
-    <!--xacro:joint_pos_transmission joint="beam_to_slider"/-->
+    <xacro:joint_transmission joint="slider_to_support"/>
     <gazebo reference="support_to_base_link">
       <provideFeedback>true</provideFeedback>
@@ -28,10 +28,10 @@
     <origin xyz="0 0 ${column_height/2}" rpy="0 0 0" />
   </joint>
-    <joint name="slider_to_support" type="prismatic">
+    <joint name="slider_to_support" type="fixed">
     <parent link="slider"/>
     <child link="support"/>
     <origin xyz="0 0 ${-1*(cross_length/2)}" rpy="0 0 0" />
-    <axis xyz="0 0 1" />
-    <limit effort="15" velocity="50" lower="0" upper="1" />
+    <axis xyz="0 1 0" />
+    <!--limit effort="3" velocity="3" lower="${-90*M_PI/180}" upper="${90*M_PI/180}" /-->
   </joint>
   <joint name="support_to_base_link" type="fixed">

Commit message: creo que los controladores estan bkn

File: urdf/leg.xacro (robot description, xacro)
@@ -192,5 +192,5 @@
     <origin xyz="0 0 ${-1*tibia_height}" rpy="0 0 0" />
     <axis xyz="0 1 0" />
-    <limit effort="8" velocity="6" lower="${-90*M_PI/180}" upper="${0*M_PI/180}" />
+    <limit effort="8" velocity="6" lower="-2.1" upper="-0.8" />
     <!--dynamics damping="${dxl_damping}" friction="${dxl_friction}" /-->
   </joint>
@@ -200,5 +200,5 @@
     <origin xyz="0 0 ${-1*ankle_height}" rpy="0 0 0" />
     <axis xyz="0 1 0" />
-    <limit effort="4" velocity="4" lower="${-45*M_PI/180}" upper="0" />
+    <limit effort="8" velocity="6" lower="${-45*M_PI/180}" upper="0" />
     <!--dynamics damping="${dxl_damping}" friction="${dxl_friction}" /-->
   </joint>

File: urdf/structure.xacro (robot description, xacro)
@@ -6,5 +6,5 @@
   <xacro:property name="cross_length" value="0.025" />
   <xacro:property name="beam_height" value="20" />
-  <xacro:property name="support_height" value="1.26" />
+  <xacro:property name="support_height" value="1.30" />
   <xacro:macro name="structure" params="parent child body_height body_width body_large">
     <xacro:joint_transmission joint="slider_to_support"/>

Commit message: asfd

File: urdf/leg.xacro (robot description, xacro)
@@ -212,5 +212,5 @@
     <parent link="${side}_ankle"/>
     <child link="${side}_phalange"/>
-    <origin xyz="0 0 ${-1*ankle_height}" rpy="0 0 0" />
+    <origin xyz="${-1*ankle_large/2} 0 ${-1*ankle_height}" rpy="0 0 0" />
     <axis xyz="0 1 0" />
     <limit effort="8" velocity="6" lower="${-45*M_PI/180}" upper="0" />

File: urdf/structure.xacro (robot description, xacro)
@@ -6,5 +6,5 @@
   <xacro:property name="cross_length" value="0.025" />
   <xacro:property name="beam_height" value="7" />
-  <xacro:property name="support_height" value="1.30" />
+  <xacro:property name="support_height" value="1.26" />
   <xacro:macro name="structure" params="parent child body_height body_width body_large">
     <xacro:joint_transmission joint="slider_to_support"/>

Commit message: nothing good

File: urdf/leg.xacro (robot description, xacro)
@@ -190,5 +190,5 @@
     <origin xyz="0 0 0" rpy="0 0 0" />
     <axis xyz="0 1 0" />
-    <limit effort="8" velocity="6" lower="${-75*M_PI/180}" upper="${45*M_PI/180}"  />
+    <limit effort="80000000" velocity="60000000" lower="${-75*M_PI/180}" upper="${45*M_PI/180}"  />
     <!--dynamics damping="${dxl_damping}" friction="${dxl_friction}" /-->
   </joint>
@@ -198,5 +198,5 @@
     <origin xyz="0 0 ${-1*thigh_height}" rpy="0 0 0" />
     <axis xyz="0 1 0" />
-    <limit effort="8" velocity="6" lower="${0*M_PI/180}" upper="${150*M_PI/180}" />
+    <limit effort="80000000" velocity="60000000" lower="${0*M_PI/180}" upper="${150*M_PI/180}" />
     <!--dynamics damping="${dxl_damping}" friction="${dxl_friction}" /-->
   </joint>
@@ -206,5 +206,5 @@
     <origin xyz="0 0 ${-1*tibia_height}" rpy="0 0 0" />
     <axis xyz="0 1 0" />
-    <limit effort="8" velocity="6" lower="-2.1" upper="-0.8" />
+    <limit effort="80000000" velocity="60000000" lower="-2.1" upper="-0.8" />
     <!--dynamics damping="${dxl_damping}" friction="${dxl_friction}" /-->
   </joint>
@@ -214,5 +214,5 @@
     <origin xyz="${-1*ankle_large/2} 0 ${-1*ankle_height}" rpy="0 0 0" />
     <axis xyz="0 1 0" />
-    <limit effort="8" velocity="6" lower="${-45*M_PI/180}" upper="0" />
+    <limit effort="80000000" velocity="60000000" lower="${-45*M_PI/180}" upper="0" />
     <!--dynamics damping="${dxl_damping}" friction="${dxl_friction}" /-->
   </joint>

File: urdf/structure.xacro (robot description, xacro)
@@ -3,5 +3,5 @@
   xmlns:xacro="http://www.ros.org/wiki/xacro"
   name="structure">
-  <xacro:property name="column_height" value="1.25" />
+  <xacro:property name="column_height" value="2" />
   <xacro:property name="cross_length" value="0.025" />
   <xacro:property name="beam_height" value="7" />
@@ -26,5 +26,5 @@
     <child link="beam"/>
     <axis xyz="0 0 1"/>
-    <origin xyz="0 0 ${column_height/2}" rpy="0 0 0" />
+    <origin xyz="0 0 0" rpy="0 0 0" />
     <limit effort="3" velocity="3" lower="1" upper="2" />
   </joint>
@@ -44,5 +44,5 @@
     <parent link="beam"/>
     <child link="slider"/>
-    <origin xyz="0 5 ${-1*cross_length}" rpy="0 0 ${90*M_PI/180}"/>
+    <origin xyz="0 0 0" rpy="0 0 ${90*M_PI/180}"/>
     <axis xyz="1 0 0" />
     <limit effort="3" velocity="2" lower="5" upper="20" />

Commit message: pff

File: urdf/leg.xacro (robot description, xacro)
@@ -212,5 +212,5 @@
     <parent link="${side}_ankle"/>
     <child link="${side}_phalange"/>
-    <origin xyz="${-1*ankle_large/2} 0 ${-1*ankle_height}" rpy="0 0 0" />
+    <origin xyz="$0 0 ${-1*ankle_height}" rpy="0 0 0" />
     <axis xyz="0 1 0" />
     <limit effort="8" velocity="6" lower="${-45*M_PI/180}" upper="0" />

File: urdf/structure.xacro (robot description, xacro)
@@ -5,16 +5,7 @@
   <xacro:property name="column_height" value="1.25" />
   <xacro:property name="cross_length" value="0.025" />
-  <xacro:property name="beam_height" value="10" />
+  <xacro:property name="beam_height" value="5" />
   <xacro:property name="support_height" value="1.26" />
   <xacro:macro name="structure" params="parent child body_height body_width body_large">
-    <xacro:joint_transmission joint="slider_to_support"/>
-    <gazebo reference="support_to_base_link">
-      <provideFeedback>true</provideFeedback>
-      <disableFixedJointLumping>true</disableFixedJointLumping>
-    </gazebo>
-      <gazebo reference="slider_to_support">
-      <provideFeedback>true</provideFeedback>
-      <disableFixedJointLumping>true</disableFixedJointLumping>
-    </gazebo>
   <joint name="fixed" type="fixed">
     <parent link="${parent}"/>
@@ -26,24 +17,11 @@
     <child link="beam"/>
     <axis xyz="0 0 1"/>
-    <origin xyz="0 0 ${column_height/2}" rpy="0 0 0" />
+    <origin xyz="0 0 ${-column_height/2}" rpy="0 0 0" />
   </joint>
-    <joint name="slider_to_support" type="fixed">
-    <parent link="slider"/>
-    <child link="support"/>
-    <origin xyz="0 0 ${-1*(cross_length/2)}" rpy="0 0 0" />
-    <axis xyz="0 1 0" />
-    <!--limit effort="3" velocity="3" lower="${-90*M_PI/180}" upper="${90*M_PI/180}" /-->
-  </joint>
-  <joint name="support_to_base_link" type="fixed">
-    <parent link="support"/>
+  <joint name="beam_to_base_link" type="fixed">
+    <parent link="beam"/>
     <child link="${child}"/>
-    <origin xyz="0 0 ${-support_height}" rpy="0 0 0" />
-  </joint>
-  <joint name="beam_to_slider" type="fixed">
-    <parent link="beam"/>
-    <child link="slider"/>
-    <origin xyz="0 1 ${-1*cross_length}" rpy="0 0 0"/>
-    <axis xyz="1 0 0" />
-    <!--limit effort="3" velocity="2" lower="5" upper="20" /-->
+    <origin xyz="0 ${beam_height} 0" rpy="0 0 0" />
+    <!--limit effort="4" velocity="4" lower="0" upper="0.01" /-->
   </joint>
   <link name="column">
@@ -64,41 +42,4 @@
       <geometry>
         <box size="${cross_length} ${cross_length} ${column_height}" />
-      </geometry>
-    </collision>
-  </link>
-    <link name="slider">
-    <inertial>
-      <origin xyz="0 0 0" />
-      <mass value="0.1"/>
-      <xacro:cuboid_inertia_def x="${cross_length}" y="${cross_length}" z="${cross_length}" mass="1"/>
-    </inertial>
-    <visual>
-      <origin xyz="0 0 0" rpy="0 0 0" />
-      <geometry>
-        <box size="${cross_length} ${cross_length} ${cross_length}" />
-      </geometry>
-    </visual>
-    <collision>
-      <geometry>
-        <box size="${cross_length} ${cross_length} ${cross_length}" />
-      </geometry>
-    </collision>
-  </link>
-    <link name="support">
-    <inertial>
-      <origin xyz="0 0 ${-1*support_height/2}" />
-      <mass value="0.4"/>
-      <xacro:cuboid_inertia_def x="${cross_length}" y="${cross_length}" z="${support_height}" mass="4"/>
-    </inertial>
-    <visual>
-      <origin xyz="0 0 ${-1*support_height/2}" rpy="0 0 0" />
-      <geometry>
-        <box size="${cross_length} ${cross_length} ${support_height}" />
-      </geometry>
-    </visual>
-    <collision>
-      <origin xyz="0 0 ${-1*support_height/2}" rpy="0 0 0" />
-      <geometry>
-        <box size="${cross_length} ${cross_length} ${support_height}" />
       </geometry>
     </collision>

Commit message: nose

File: urdf/leg.xacro (robot description, xacro)
@@ -44,5 +44,5 @@
   <link name="${side}_pelvis" >
     <inertial>
-      <origin xyz="0 0 ${-1*pelvis_height/2}" />
+      <origin xyz="0 0 0" />
       <mass value="0.2"/>
       <xacro:cuboid_inertia_def x="${pelvis_large}" y="${pelvis_width}" z="${pelvis_height}" mass="0.2"/>
@@ -81,5 +81,5 @@
   <link name="${side}_thigh" >
     <inertial>
-      <origin xyz="0 0 ${-1*thigh_height/2}" />
+      <origin xyz="0 0 0" />
       <mass value="0.25"/>
       <xacro:cuboid_inertia_def x="${thigh_large}" y="${thigh_width}" z="${thigh_height}" mass="0.5"/>
@@ -100,5 +100,5 @@
   <link name="${side}_tibia" >
     <inertial>
-      <origin xyz="0 0 ${-1*tibia_height/2}" />
+      <origin xyz="0 0 0" />
       <mass value="0.2"/>
       <xacro:cuboid_inertia_def x="${tibia_large}" y="${tibia_width}" z="${tibia_height}" mass="0.4"/>
@@ -119,5 +119,5 @@
   <link name="${side}_ankle" >
     <inertial>
-      <origin xyz="0 0 ${-1*ankle_height/2}" />
+      <origin xyz="0 0 0" />
       <mass value="0.2"/>
       <xacro:cuboid_inertia_def x="${ankle_large}" y="${ankle_width}" z="${ankle_height}" mass="0.2"/>
@@ -144,5 +144,5 @@
   <link name="${side}_phalange" >
     <inertial>
-      <origin xyz="0 0 ${-1*phalange_height/2}" />
+      <origin xyz="0 0 0" />
       <mass value="0.07"/>
       <xacro:cuboid_inertia_def x="${phalange_large}" y="${phalange_width}" z="${phalange_height}" mass="0.07"/>

Commit message: camina un poco

File: urdf/leg.xacro (robot description, xacro)
@@ -19,6 +19,6 @@
  <xacro:property name="tibia_large" value="0.045" />
   <xacro:property name="ankle_height" value="0.0745" />
- <xacro:property name="ankle_width" value="0.035" />
- <xacro:property name="ankle_large" value="0.045" />
+ <xacro:property name="ankle_width" value="0.020" />
+ <xacro:property name="ankle_large" value="0.020" />
    <xacro:property name="phalange_height" value="0.0745" />
  <xacro:property name="phalange_width" value="0.020" />

Commit message: algo camina

File: urdf/leg.xacro (robot description, xacro)
@@ -21,12 +21,12 @@
  <xacro:property name="ankle_width" value="0.020" />
  <xacro:property name="ankle_large" value="0.020" />
-   <xacro:property name="phalange_height" value="0.0745" />
+   <xacro:property name="phalange_height" value="0.1" />
  <xacro:property name="phalange_width" value="0.020" />
  <xacro:property name="phalange_large" value="0.020" />
    <!-- Friction model from "Characterization and modeling of a Dynamixel servo" by Arno Mensin (model AX12, better than nothing) -->
   <!-- Damping N.m.s/rad -->
-  <xacro:property name="dxl_damping" value="0.15" />
+  <xacro:property name="dxl_damping" value="0.85" />
   <!-- Friccion N.m -->
-  <xacro:property name="dxl_friction" value="0.3" />
+  <xacro:property name="dxl_friction" value="0.9" />
   <xacro:macro name="cuboid_inertia_def" params="x y z mass">
     <inertia
@@ -144,7 +144,7 @@
   <link name="${side}_phalange" >
     <inertial>
-      <origin xyz="0 0 0" />
-      <mass value="0.07"/>
-      <xacro:cuboid_inertia_def x="${phalange_large}" y="${phalange_width}" z="${phalange_height}" mass="0.07"/>
+      <origin xyz="0 0 ${-1*phalange_height/2}" />
+      <mass value="2"/>
+      <xacro:cuboid_inertia_def x="${phalange_large}" y="${phalange_width}" z="${phalange_height}" mass="2"/>
     </inertial>
     <visual>
@@ -175,5 +175,5 @@
     <axis xyz="0 0 1" />
     <!--limit effort="4" velocity="4" lower="0" upper="0.01" /-->
-    <!--dynamics damping="${dxl_damping}" friction="${dxl_friction}" /-->
+    <dynamics damping="${dxl_damping}" friction="${dxl_friction}" />
   </joint>
   <joint name="${side}_thigh_yaw_joint" type="fixed">
@@ -191,5 +191,5 @@
     <axis xyz="0 1 0" />
     <limit effort="8" velocity="6" lower="${-75*M_PI/180}" upper="${45*M_PI/180}"  />
-    <!--dynamics damping="${dxl_damping}" friction="${dxl_friction}" /-->
+    <dynamics damping="${dxl_damping}" friction="${dxl_friction}" />
   </joint>
   <joint name="${side}_tibia_joint" type="revolute">
@@ -199,5 +199,5 @@
     <axis xyz="0 1 0" />
     <limit effort="8" velocity="6" lower="${0*M_PI/180}" upper="${150*M_PI/180}" />
-    <!--dynamics damping="${dxl_damping}" friction="${dxl_friction}" /-->
+    <dynamics damping="${dxl_damping}" friction="${dxl_friction}" />
   </joint>
   <joint name="${side}_ankle_joint" type="revolute">
@@ -207,5 +207,5 @@
     <axis xyz="0 1 0" />
     <limit effort="8" velocity="6" lower="-2.1" upper="-0.8" />
-    <!--dynamics damping="${dxl_damping}" friction="${dxl_friction}" /-->
+    <dynamics damping="${dxl_damping}" friction="${dxl_friction}" />
   </joint>
   <joint name="${side}_phalange_joint" type="revolute">
@@ -215,5 +215,5 @@
     <axis xyz="0 1 0" />
     <limit effort="8" velocity="6" lower="${-45*M_PI/180}" upper="0" />
-    <!--dynamics damping="${dxl_damping}" friction="${dxl_friction}" /-->
+    <dynamics damping="${dxl_damping}" friction="${dxl_friction}" />
   </joint>
 </xacro:macro>

Commit message: no camina pero no explota

File: urdf/leg.xacro (robot description, xacro)
@@ -21,12 +21,12 @@
  <xacro:property name="ankle_width" value="0.020" />
  <xacro:property name="ankle_large" value="0.020" />
-   <xacro:property name="phalange_height" value="0.1" />
+   <xacro:property name="phalange_height" value="0.08" />
  <xacro:property name="phalange_width" value="0.020" />
  <xacro:property name="phalange_large" value="0.020" />
    <!-- Friction model from "Characterization and modeling of a Dynamixel servo" by Arno Mensin (model AX12, better than nothing) -->
   <!-- Damping N.m.s/rad -->
-  <xacro:property name="dxl_damping" value="0.85" />
+  <xacro:property name="dxl_damping" value="0.5" />
   <!-- Friccion N.m -->
-  <xacro:property name="dxl_friction" value="0.9" />
+  <xacro:property name="dxl_friction" value="0.5" />
   <xacro:macro name="cuboid_inertia_def" params="x y z mass">
     <inertia
@@ -145,6 +145,6 @@
     <inertial>
       <origin xyz="0 0 ${-1*phalange_height/2}" />
-      <mass value="2"/>
-      <xacro:cuboid_inertia_def x="${phalange_large}" y="${phalange_width}" z="${phalange_height}" mass="2"/>
+      <mass value="0.15"/>
+      <xacro:cuboid_inertia_def x="${phalange_large}" y="${phalange_width}" z="${phalange_height}" mass="0.15"/>
     </inertial>
     <visual>
@@ -159,5 +159,5 @@
         <box size="${phalange_large} ${phalange_width} ${phalange_height}"/>
       </geometry>
-       <surface>
+       <!--surface>
         <friction>
           <ode>
@@ -166,5 +166,5 @@
           </ode>
         </friction>
-      </surface>
+      </surface-->
     </collision>
   </link>
@@ -215,5 +215,5 @@
     <axis xyz="0 1 0" />
     <limit effort="8" velocity="6" lower="${-45*M_PI/180}" upper="0" />
-    <dynamics damping="${dxl_damping}" friction="${dxl_friction}" />
+    <!--dynamics damping="${dxl_damping}" friction="${dxl_friction}" /-->
   </joint>
 </xacro:macro>

Commit message: camina con buenas inercias

File: urdf/leg.xacro (robot description, xacro)
@@ -44,5 +44,5 @@
   <link name="${side}_pelvis" >
     <inertial>
-      <origin xyz="0 0 0" />
+      <origin xyz="0 0 ${-1*pelvis_height/2}" />
       <mass value="0.2"/>
       <xacro:cuboid_inertia_def x="${pelvis_large}" y="${pelvis_width}" z="${pelvis_height}" mass="0.2"/>
@@ -81,5 +81,5 @@
   <link name="${side}_thigh" >
     <inertial>
-      <origin xyz="0 0 0" />
+      <origin xyz="0 0 ${-1*thigh_height/2}" />
       <mass value="0.25"/>
       <xacro:cuboid_inertia_def x="${thigh_large}" y="${thigh_width}" z="${thigh_height}" mass="0.5"/>
@@ -100,5 +100,5 @@
   <link name="${side}_tibia" >
     <inertial>
-      <origin xyz="0 0 0" />
+      <origin xyz="0 0 ${-1*tibia_height/2}" />
       <mass value="0.2"/>
       <xacro:cuboid_inertia_def x="${tibia_large}" y="${tibia_width}" z="${tibia_height}" mass="0.4"/>
@@ -119,5 +119,5 @@
   <link name="${side}_ankle" >
     <inertial>
-      <origin xyz="0 0 0" />
+      <origin xyz="0 0 ${-1*ankle_height/2}" />
       <mass value="0.2"/>
       <xacro:cuboid_inertia_def x="${ankle_large}" y="${ankle_width}" z="${ankle_height}" mass="0.2"/>

Commit message: casi

File: urdf/leg.xacro (robot description, xacro)
@@ -82,5 +82,5 @@
     <inertial>
       <origin xyz="0 0 ${-1*thigh_height/2}" />
-      <mass value="0.25"/>
+      <mass value="0.20"/>
       <xacro:cuboid_inertia_def x="${thigh_large}" y="${thigh_width}" z="${thigh_height}" mass="0.5"/>
     </inertial>
@@ -101,6 +101,6 @@
     <inertial>
       <origin xyz="0 0 ${-1*tibia_height/2}" />
-      <mass value="0.2"/>
-      <xacro:cuboid_inertia_def x="${tibia_large}" y="${tibia_width}" z="${tibia_height}" mass="0.4"/>
+      <mass value="0.35"/>
+      <xacro:cuboid_inertia_def x="${tibia_large}" y="${tibia_width}" z="${tibia_height}" mass="0.35"/>
     </inertial>
     <visual>
@@ -120,6 +120,6 @@
     <inertial>
       <origin xyz="0 0 ${-1*ankle_height/2}" />
-      <mass value="0.2"/>
-      <xacro:cuboid_inertia_def x="${ankle_large}" y="${ankle_width}" z="${ankle_height}" mass="0.2"/>
+      <mass value="0.05"/>
+      <xacro:cuboid_inertia_def x="${ankle_large}" y="${ankle_width}" z="${ankle_height}" mass="0.05"/>
     </inertial>
     <visual>
@@ -145,6 +145,6 @@
     <inertial>
       <origin xyz="0 0 ${-1*phalange_height/2}" />
-      <mass value="0.15"/>
-      <xacro:cuboid_inertia_def x="${phalange_large}" y="${phalange_width}" z="${phalange_height}" mass="0.15"/>
+      <mass value="0.06"/>
+      <xacro:cuboid_inertia_def x="${phalange_large}" y="${phalange_width}" z="${phalange_height}" mass="0.06"/>
     </inertial>
     <visual>
