Commit message: add slide

File: urdf/details.xacro (robot description, xacro)
@@ -35,5 +35,5 @@
     <inertial>
       <origin xyz="-0.003053 -0.038651 -0.019268" />
-      <mass value="0.97559947"/>
+      <mass value="5"/>
       <inertia ixx="3.1081800"  ixy="-0.25460189"  ixz="2.0318174" iyy="6.3787776" iyz="0.16417863" izz="5.3316425" />
     </inertial>

File: urdf/structure.xacro (robot description, xacro)
@@ -3,8 +3,8 @@
   xmlns:xacro="http://www.ros.org/wiki/xacro"
   name="structure">
-  <xacro:property name="column_height" value="1.06" />
+  <xacro:property name="column_height" value="1.25" />
   <xacro:property name="cross_length" value="0.025" />
-  <xacro:property name="beam_height" value="1.006" />
-  <xacro:property name="support_height" value="1.205" />
+  <xacro:property name="beam_height" value="10" />
+  <xacro:property name="support_height" value="0.25" />
   <xacro:macro name="structure" params="parent child body_height body_width body_large">
   <joint name="fixed" type="fixed">
@@ -13,5 +13,5 @@
     <origin xyz="0 0 0" rpy="0 0 0" />
   </joint>
-  <joint name="column_to_beam" type="continuous">
+  <joint name="column_to_beam" type="fixed">
     <parent link="column"/>
     <child link="beam"/>
@@ -19,8 +19,10 @@
     <origin xyz="0 0 ${column_height/2}" rpy="0 0 0" />
   </joint>
-    <joint name="beam_to_support" type="fixed">
-    <parent link="beam"/>
+    <joint name="slider_to_support" type="revolute">
+    <parent link="slider"/>
     <child link="support"/>
-    <origin xyz="0 ${beam_height} ${-1*support_height/2}" rpy="0 0 0" />
+    <origin xyz="0 0 0" rpy="0 0 0" />
+    <axis xyz="0 1 0" />
+    <limit effort="10" velocity="5.6548668" lower="${-90*M_PI/180}" upper="${90*M_PI/180}" />
   </joint>
   <joint name="support_to_base_link" type="fixed">
@@ -28,4 +30,11 @@
     <child link="${child}"/>
     <origin xyz="0 0 ${-1*support_height/2}" rpy="0 0 0" />
+  </joint>
+  <joint name="beam_to_slider" type="prismatic">
+    <parent link="beam"/>
+    <child link="slider"/>
+    <origin xyz="0 0 0" rpy="0 0 0" />
+    <axis xyz="0 1 0" />
+    <limit effort="10" velocity="5.6548668" lower="0" upper="5" />
   </joint>
   <link name="column">
@@ -48,4 +57,5 @@
     </collision>
   </link>
+    <link name="slider"/>
     <link name="support">
     <inertial>

Commit message: changes to inertias

File: urdf/details.xacro (robot description, xacro)
@@ -6,7 +6,7 @@
  <link name="neck">
     <inertial>
-      <origin xyz="-0.003053 -0.038651 -0.019268" />
-      <mass value="0.97559947"/>
-      <inertia ixx="3.1081800"  ixy="-0.25460189"  ixz="2.0318174" iyy="6.3787776" iyz="0.16417863" izz="5.3316425" />
+      <origin xyz="0 0 0" />
+      <mass value="0.01"/>
+      <xacro:cuboid_inertia_def x="${body_large/7}" y="${body_width/7}" z="${body_height/7}" mass="0.01"/>
     </inertial>
     <visual>
@@ -20,7 +20,7 @@
     <link name="head">
     <inertial>
-      <origin xyz="-0.003053 -0.038651 -0.019268" />
-      <mass value="0.97559947"/>
-      <inertia ixx="3.1081800"  ixy="-0.25460189"  ixz="2.0318174" iyy="6.3787776" iyz="0.16417863" izz="5.3316425" />
+      <origin xyz="0 0 0" />
+      <mass value="0.5"/>
+      <xacro:cuboid_inertia_def x="${body_large/2}" y="${body_width*0.8}" z="${body_height*0.6}" mass="0.5"/>
     </inertial>
     <visual>
@@ -34,7 +34,7 @@
   <link name="tail">
     <inertial>
-      <origin xyz="-0.003053 -0.038651 -0.019268" />
-      <mass value="5"/>
-      <inertia ixx="3.1081800"  ixy="-0.25460189"  ixz="2.0318174" iyy="6.3787776" iyz="0.16417863" izz="5.3316425" />
+      <origin xyz="0 0 0" />
+      <mass value="0.6"/>
+      <xacro:cuboid_inertia_def x="${body_large*2}" y="${body_width}" z="${body_height/2}" mass="0.6"/>
     </inertial>
     <visual>

File: urdf/experiment.xacro (robot description, xacro)
@@ -17,7 +17,7 @@
   <link name="body">
     <inertial>
-      <origin xyz="-0.003053 -0.038651 -0.019268" />
-      <mass value="0.97559947"/>
-      <inertia ixx="3.1081800"  ixy="-0.25460189"  ixz="2.0318174" iyy="6.3787776" iyz="0.16417863" izz="5.3316425" />
+      <origin xyz="0 0 0" />
+      <mass value="0.8"/>
+      <xacro:cuboid_inertia_def x="${body_large}" y="${body_width}" z="${body_height}" mass="0.8"/>
     </inertial>
     <visual>

File: urdf/leg.xacro (robot description, xacro)
@@ -24,17 +24,24 @@
  <xacro:property name="phalange_width" value="0.020" />
  <xacro:property name="phalange_large" value="0.020" />
+  <xacro:macro name="cuboid_inertia_def" params="x y z mass">
+    <inertia
+      iyy="${mass*(z*z+x*x)/12.0}"
+      ixx="${mass*(y*y+z*z)/12.0}"
+      izz="${mass*(x*x+y*y)/12.0}"
+      ixy="0.0" iyz="0.0" ixz="0.0"/>
+  </xacro:macro>
   <xacro:macro name="leg" params="side parent reflect body_height body_width body_large">
       <!-- Transmissions -->
-    <xacro:joint_pos_transmission joint="${side}_pelvis_joint"/>
-    <xacro:joint_pos_transmission joint="${side}_thigh_yaw_joint"/>
-    <xacro:joint_pos_transmission joint="${side}_thigh_pitch_joint"/>
-    <xacro:joint_pos_transmission joint="${side}_tibia_joint"/>
-    <xacro:joint_pos_transmission joint="${side}_ankle_joint"/>
-    <xacro:joint_pos_transmission joint="${side}_phalange_joint"/>
+    <xacro:joint_transmission joint="${side}_pelvis_joint"/>
+    <xacro:joint_transmission joint="${side}_thigh_yaw_joint"/>
+    <xacro:joint_transmission joint="${side}_thigh_pitch_joint"/>
+    <xacro:joint_transmission joint="${side}_tibia_joint"/>
+    <xacro:joint_transmission joint="${side}_ankle_joint"/>
+    <xacro:joint_transmission joint="${side}_phalange_joint"/>
   <link name="${side}_pelvis" >
     <inertial>
-      <origin xyz="0.000000 0.000480 0.018437" />
-      <mass value="0.167"/>
-      <inertia ixx="0.12259691"  ixy="0.00071127469"  ixz="0.00081143913" iyx="0.00071127469" iyy="0.11066637" iyz="-0.0071635476" izx="0.00081143913" izy="-0.0071635476" izz="0.041877668" />
+      <origin xyz="0 0 0" />
+      <mass value="0.1"/>
+      <xacro:cuboid_inertia_def x="${pelvis_large}" y="${pelvis_width}" z="${pelvis_height}" mass="0.2"/>
     </inertial>
     <visual>
@@ -53,7 +60,7 @@
   <link name="${side}_thigh_yaw" >
     <inertial>
-      <origin xyz="0.000079 0.018242 0.013873" />
-      <mass value="0.11904336"/>
-      <inertia ixx="0.097950272"  ixy="0.0012119368"  ixz="-0.00021223016" iyx="0.00122119368" iyy="0.032848287" iyz="-0.0019474021" izx="-0.00021223016" izy="-0.0019474021" izz="0.11493509" />
+      <origin xyz="0 0 0" />
+      <mass value="0.01"/>
+      <xacro:cuboid_inertia_def x="${thigh_virtual_large}" y="${thigh_virtual_width}" z="${thigh_virtual_height}" mass="0.2"/>
     </inertial>
     <visual>
@@ -71,7 +78,7 @@
   <link name="${side}_thigh" >
     <inertial>
-      <origin xyz="-0.062965 -0.000323 0.000692" />
-      <mass value="0.11904336"/>
-      <inertia ixx="0.097950272"  ixy="0.0012119368"  ixz="-0.00021223016" iyx="0.00122119368" iyy="0.032848287" iyz="-0.0019474021" izx="-0.00021223016" izy="-0.0019474021" izz="0.11493509" />
+      <origin xyz="0 0 0" />
+      <mass value="0.2"/>
+      <xacro:cuboid_inertia_def x="${thigh_large}" y="${thigh_width}" z="${thigh_height}" mass="0.2"/>
     </inertial>
     <visual>
@@ -90,7 +97,7 @@
   <link name="${side}_tibia" >
     <inertial>
-      <origin xyz="-0.053955 0.006548 -0.000592" />
-      <mass value="0.070309794"/>
-      <inertia ixx="0.093369608"  ixy="-0.00093567395"  ixz="-0.00023992085" iyx="-0.00093567395" iyy="0.046295534" iyz="-0.012858493" izx="-0.00023992085" izy="-0.012858493" izz="0.11351516" />
+      <origin xyz="0 0 0" />
+      <mass value="0.15"/>
+      <xacro:cuboid_inertia_def x="${tibia_large}" y="${tibia_width}" z="${tibia_height}" mass="0.2"/>
     </inertial>
     <visual>
@@ -109,7 +116,7 @@
   <link name="${side}_ankle" >
     <inertial>
-      <origin xyz="-0.000214 -0.018536 0.013873" />
-      <mass value="0.16710792"/>
-      <inertia ixx="0.12079175"  ixy="-0.00079781067"  ixz="-0.00039322246" iyx="-0.00079781067" iyy="0.10885465" iyz="0.0070770117" izx="-0.00039322246" izy="0.0070770117" izz="0.041871103" />
+      <origin xyz="0 0 0" />
+      <mass value="0.1"/>
+      <xacro:cuboid_inertia_def x="${ankle_large}" y="${ankle_width}" z="${ankle_height}" mass="0.2"/>
     </inertial>
     <visual>
@@ -128,7 +135,7 @@
   <link name="${side}_phalange" >
     <inertial>
-      <origin xyz="-0.000214 -0.018536 0.013873" />
-      <mass value="0.16710792"/>
-      <inertia ixx="0.12079175"  ixy="-0.00079781067"  ixz="-0.00039322246" iyx="-0.00079781067" iyy="0.10885465" iyz="0.0070770117" izx="-0.00039322246" izy="0.0070770117" izz="0.041871103" />
+      <origin xyz="0 0 0" />
+      <mass value="0.05"/>
+      <xacro:cuboid_inertia_def x="${phalange_large}" y="${phalange_width}" z="${phalange_height}" mass="0.2"/>
     </inertial>
     <visual>

File: urdf/structure.xacro (robot description, xacro)
@@ -6,5 +6,5 @@
   <xacro:property name="cross_length" value="0.025" />
   <xacro:property name="beam_height" value="10" />
-  <xacro:property name="support_height" value="0.80" />
+  <xacro:property name="support_height" value="1.30" />
   <xacro:macro name="structure" params="parent child body_height body_width body_large">
   <joint name="fixed" type="fixed">
@@ -22,5 +22,5 @@
     <parent link="slider"/>
     <child link="support"/>
-    <origin xyz="0 0 0" rpy="0 0 0" />
+    <origin xyz="0 0 ${-1*(cross_length/2)}" rpy="0 0 0" />
     <axis xyz="0 1 0" />
     <limit effort="10" velocity="5.6548668" lower="${-90*M_PI/180}" upper="${90*M_PI/180}" />
@@ -29,18 +29,18 @@
     <parent link="support"/>
     <child link="${child}"/>
-    <origin xyz="0 0 ${-1*support_height/2}" rpy="0 0 0" />
+    <origin xyz="0 0 ${-support_height}" rpy="0 0 0" />
   </joint>
   <joint name="beam_to_slider" type="prismatic">
     <parent link="beam"/>
     <child link="slider"/>
-    <origin xyz="0 0 0" rpy="0 0 ${90*M_PI/180}" />
+    <origin xyz="0 0 ${-1*cross_length}" rpy="0 0 ${90*M_PI/180}" />
     <axis xyz="1 0 0" />
-    <limit effort="10" velocity="5.6548668" lower="3" upper="15" />
+    <limit effort="100" velocity="50.6548668" lower="3" upper="15" />
   </joint>
   <link name="column">
     <inertial>
-      <origin xyz="-0.003053 -0.038651 -0.019268" />
-      <mass value="0.97559947"/>
-      <inertia ixx="3.1081800"  ixy="-0.25460189"  ixz="2.0318174" iyy="6.3787776" iyz="0.16417863" izz="5.3316425" />
+      <origin xyz="0 0 0" />
+      <mass value="0.8"/>
+      <xacro:cuboid_inertia_def x="${cross_length}" y="${cross_length}" z="${column_height}" mass="0.8"/>
     </inertial>
     <visual>
@@ -59,7 +59,7 @@
     <link name="slider">
     <inertial>
-      <origin xyz="-0.003053 -0.038651 -0.019268" />
-      <mass value="0.97559947"/>
-      <inertia ixx="3.1081800"  ixy="-0.25460189"  ixz="2.0318174" iyy="6.3787776" iyz="0.16417863" izz="5.3316425" />
+      <origin xyz="0 0 0" />
+      <mass value="0.1"/>
+      <xacro:cuboid_inertia_def x="${cross_length}" y="${cross_length}" z="${cross_length}" mass="0.1"/>
     </inertial>
     <visual>
@@ -77,10 +77,10 @@
     <link name="support">
     <inertial>
-      <origin xyz="-0.003053 -0.038651 -0.019268" />
-      <mass value="0.97559947"/>
-      <inertia ixx="3.1081800"  ixy="-0.25460189"  ixz="2.0318174" iyy="6.3787776" iyz="0.16417863" izz="5.3316425" />
+      <origin xyz="0 0 ${-1*support_height/2}" />
+      <mass value="0.8"/>
+      <xacro:cuboid_inertia_def x="${cross_length}" y="${cross_length}" z="${support_height}" mass="0.8"/>
     </inertial>
     <visual>
-      <origin xyz="0 0 0" rpy="0 0 0" />
+      <origin xyz="0 0 ${-1*support_height/2}" rpy="0 0 0" />
       <geometry>
         <box size="${cross_length} ${cross_length} ${support_height}" />
@@ -88,4 +88,5 @@
     </visual>
     <collision>
+      <origin xyz="0 0 ${-1*support_height/2}" rpy="0 0 0" />
       <geometry>
         <box size="${cross_length} ${cross_length} ${support_height}" />
@@ -95,7 +96,7 @@
     <link name="beam">
     <inertial>
-      <origin xyz="-0.003053 -0.038651 -0.019268" />
-      <mass value="0.97559947"/>
-      <inertia ixx="3.1081800"  ixy="-0.25460189"  ixz="2.0318174" iyy="6.3787776" iyz="0.16417863" izz="5.3316425" />
+      <origin xyz="0 ${beam_height/2} 0" />
+      <mass value="0.8"/>
+      <xacro:cuboid_inertia_def x="${cross_length}" y="${beam_height}" z="${cross_length}" mass="0.8"/>
     </inertial>
     <visual>

Commit message: now works

File: urdf/details.xacro (robot description, xacro)
@@ -17,4 +17,11 @@
       </geometry>
     </visual>
+    <collision>
+      <origin xyz="0 0 0" rpy="0 0 0" />
+      <!--origin xyz="-0.0235 0 -0.03525" rpy="0 0 0" /-->
+      <geometry>
+        <box size="${body_large/7} ${body_width/7} ${body_height/7}" />
+      </geometry>
+    </collision>
   </link>
     <link name="head">
@@ -31,4 +38,11 @@
       </geometry>
     </visual>
+    <collision>
+      <origin xyz="${body_large*0.5/2} 0 0" rpy="0 0 0" />
+      <!--origin xyz="-0.0235 0 -0.03525" rpy="0 0 0" /-->
+      <geometry>
+        <box size="${body_large*0.5} ${body_width*0.8} ${body_height*0.6}" />
+      </geometry>
+    </collision>
   </link>
   <link name="tail">
@@ -45,4 +59,11 @@
       </geometry>
     </visual>
+    <collision>
+      <origin xyz="-0.250 0 0" rpy="0 ${-M_PI/2} 0" />
+      <!--origin xyz="-0.0235 0 -0.03525" rpy="0 0 0" /-->
+      <geometry>
+        <mesh filename="package://simple_biped/cone.stl" scale="0.005 0.005 0.005"/>
+      </geometry>
+    </collision>
   </link>
   <joint name="body_to_tail" type="fixed">

File: urdf/leg.xacro (robot description, xacro)
@@ -43,5 +43,5 @@
       <origin xyz="0 0 0" />
       <mass value="0.1"/>
-      <xacro:cuboid_inertia_def x="${pelvis_large}" y="${pelvis_width}" z="${pelvis_height}" mass="0.2"/>
+      <xacro:cuboid_inertia_def x="${pelvis_large}" y="${pelvis_width}" z="${pelvis_height}" mass="100"/>
     </inertial>
     <visual>
@@ -62,5 +62,5 @@
       <origin xyz="0 0 0" />
       <mass value="0.01"/>
-      <xacro:cuboid_inertia_def x="${thigh_virtual_large}" y="${thigh_virtual_width}" z="${thigh_virtual_height}" mass="0.2"/>
+      <xacro:cuboid_inertia_def x="${thigh_virtual_large}" y="${thigh_virtual_width}" z="${thigh_virtual_height}" mass="100"/>
     </inertial>
     <visual>
@@ -80,5 +80,5 @@
       <origin xyz="0 0 0" />
       <mass value="0.2"/>
-      <xacro:cuboid_inertia_def x="${thigh_large}" y="${thigh_width}" z="${thigh_height}" mass="0.2"/>
+      <xacro:cuboid_inertia_def x="${thigh_large}" y="${thigh_width}" z="${thigh_height}" mass="100"/>
     </inertial>
     <visual>
@@ -99,5 +99,5 @@
       <origin xyz="0 0 0" />
       <mass value="0.15"/>
-      <xacro:cuboid_inertia_def x="${tibia_large}" y="${tibia_width}" z="${tibia_height}" mass="0.2"/>
+      <xacro:cuboid_inertia_def x="${tibia_large}" y="${tibia_width}" z="${tibia_height}" mass="100"/>
     </inertial>
     <visual>
@@ -118,5 +118,5 @@
       <origin xyz="0 0 0" />
       <mass value="0.1"/>
-      <xacro:cuboid_inertia_def x="${ankle_large}" y="${ankle_width}" z="${ankle_height}" mass="0.2"/>
+      <xacro:cuboid_inertia_def x="${ankle_large}" y="${ankle_width}" z="${ankle_height}" mass="100"/>
     </inertial>
     <visual>
@@ -137,5 +137,5 @@
       <origin xyz="0 0 0" />
       <mass value="0.05"/>
-      <xacro:cuboid_inertia_def x="${phalange_large}" y="${phalange_width}" z="${phalange_height}" mass="0.2"/>
+      <xacro:cuboid_inertia_def x="${phalange_large}" y="${phalange_width}" z="${phalange_height}" mass="100"/>
     </inertial>
     <visual>

File: urdf/structure.xacro (robot description, xacro)
@@ -42,5 +42,5 @@
       <origin xyz="0 0 0" />
       <mass value="0.8"/>
-      <xacro:cuboid_inertia_def x="${cross_length}" y="${cross_length}" z="${column_height}" mass="0.8"/>
+      <xacro:cuboid_inertia_def x="${cross_length}" y="${cross_length}" z="${column_height}" mass="100000"/>
     </inertial>
     <visual>
@@ -52,4 +52,5 @@
     </visual>
     <collision>
+      <origin xyz="0 0 0" rpy="0 0 0" />
       <geometry>
         <box size="${cross_length} ${cross_length} ${column_height}" />
@@ -61,5 +62,5 @@
       <origin xyz="0 0 0" />
       <mass value="0.1"/>
-      <xacro:cuboid_inertia_def x="${cross_length}" y="${cross_length}" z="${cross_length}" mass="0.1"/>
+      <xacro:cuboid_inertia_def x="${cross_length}" y="${cross_length}" z="${cross_length}" mass="100000"/>
     </inertial>
     <visual>
@@ -79,5 +80,5 @@
       <origin xyz="0 0 ${-1*support_height/2}" />
       <mass value="0.8"/>
-      <xacro:cuboid_inertia_def x="${cross_length}" y="${cross_length}" z="${support_height}" mass="0.8"/>
+      <xacro:cuboid_inertia_def x="${cross_length}" y="${cross_length}" z="${support_height}" mass="100"/>
     </inertial>
     <visual>
@@ -98,5 +99,5 @@
       <origin xyz="0 ${beam_height/2} 0" />
       <mass value="0.8"/>
-      <xacro:cuboid_inertia_def x="${cross_length}" y="${beam_height}" z="${cross_length}" mass="0.8"/>
+      <xacro:cuboid_inertia_def x="${cross_length}" y="${beam_height}" z="${cross_length}" mass="100000"/>
     </inertial>
     <visual>
@@ -108,4 +109,5 @@
     </visual>
     <collision>
+      <origin xyz="0 ${beam_height/2} 0" rpy="0 0 0" />
       <geometry>
         <box size="${cross_length} ${beam_height} ${cross_length} " />

Commit message: inercias buenas pero no camina

File: urdf/details.xacro (robot description, xacro)
@@ -4,4 +4,16 @@
   name="details">
   <xacro:macro name="details" params="parent body_height body_width body_large">
+ <gazebo reference="body_to_tail">
+      <provideFeedback>true</provideFeedback>
+      <disableFixedJointLumping>true</disableFixedJointLumping>
+    </gazebo>
+   <gazebo reference="neck_to_head">
+      <provideFeedback>true</provideFeedback>
+      <disableFixedJointLumping>true</disableFixedJointLumping>
+    </gazebo>
+    <gazebo reference="body_to_neck">
+      <provideFeedback>true</provideFeedback>
+      <disableFixedJointLumping>true</disableFixedJointLumping>
+    </gazebo>
  <link name="neck">
     <inertial>
@@ -27,5 +39,5 @@
     <link name="head">
     <inertial>
-      <origin xyz="0 0 0" />
+      <origin xyz="${body_large/4} 0 0" />
       <mass value="0.5"/>
       <xacro:cuboid_inertia_def x="${body_large/2}" y="${body_width*0.8}" z="${body_height*0.6}" mass="0.5"/>
@@ -48,5 +60,5 @@
   <link name="tail">
     <inertial>
-      <origin xyz="0 0 0" />
+      <origin xyz="-0.200 0 0" />
       <mass value="0.6"/>
       <xacro:cuboid_inertia_def x="${body_large*2}" y="${body_width}" z="${body_height/2}" mass="0.6"/>

File: urdf/experiment.xacro (robot description, xacro)
@@ -9,5 +9,4 @@
  <xacro:property name="body_width" value="0.100" />
  <xacro:property name="body_large" value="0.250" />
-<disableFixedJointLumping>true</disableFixedJointLumping>
   <link name="world"/>
   <link name="base_link"/>

File: urdf/leg.xacro (robot description, xacro)
@@ -44,5 +44,5 @@
   <link name="${side}_pelvis" >
     <inertial>
-      <origin xyz="0 0 0" />
+      <origin xyz="0 0 ${-1*pelvis_height/2}" />
       <mass value="0.3"/>
       <xacro:cuboid_inertia_def x="${pelvis_large}" y="${pelvis_width}" z="${pelvis_height}" mass="0.3"/>
@@ -81,5 +81,5 @@
   <link name="${side}_thigh" >
     <inertial>
-      <origin xyz="0 0 0" />
+      <origin xyz="0 0 ${-1*thigh_height/2}" />
       <mass value="0.8"/>
       <xacro:cuboid_inertia_def x="${thigh_large}" y="${thigh_width}" z="${thigh_height}" mass="0.8"/>
@@ -100,5 +100,5 @@
   <link name="${side}_tibia" >
     <inertial>
-      <origin xyz="0 0 0" />
+      <origin xyz="0 0 ${-1*tibia_height/2}" />
       <mass value="0.6"/>
       <xacro:cuboid_inertia_def x="${tibia_large}" y="${tibia_width}" z="${tibia_height}" mass="0.6"/>
@@ -119,5 +119,5 @@
   <link name="${side}_ankle" >
     <inertial>
-      <origin xyz="0 0 0" />
+      <origin xyz="0 0 ${-1*ankle_height/2}" />
       <mass value="0.3"/>
       <xacro:cuboid_inertia_def x="${ankle_large}" y="${ankle_width}" z="${ankle_height}" mass="0.3"/>
@@ -138,5 +138,5 @@
   <link name="${side}_phalange" >
     <inertial>
-      <origin xyz="0 0 0" />
+      <origin xyz="0 0 ${-1*phalange_height/2}" />
       <mass value="0.1"/>
       <xacro:cuboid_inertia_def x="${phalange_large}" y="${phalange_width}" z="${phalange_height}" mass="0.1"/>

File: urdf/structure.xacro (robot description, xacro)
@@ -8,4 +8,8 @@
   <xacro:property name="support_height" value="1.30" />
   <xacro:macro name="structure" params="parent child body_height body_width body_large">
+    <gazebo reference="support_to_base_link">
+      <provideFeedback>true</provideFeedback>
+      <disableFixedJointLumping>true</disableFixedJointLumping>
+    </gazebo>
   <joint name="fixed" type="fixed">
     <parent link="${parent}"/>
