Commit message: doesnt work

File: urdf/details.xacro (robot description, xacro)
@@ -8,8 +8,8 @@
       <disableFixedJointLumping>true</disableFixedJointLumping>
     </gazebo>
-   <gazebo reference="neck_to_head">
+   <!--gazebo reference="neck_to_head">
       <provideFeedback>true</provideFeedback>
       <disableFixedJointLumping>true</disableFixedJointLumping>
-    </gazebo>
+    </gazebo-->
     <gazebo reference="body_to_neck">
       <provideFeedback>true</provideFeedback>

File: urdf/structure.xacro (robot description, xacro)
@@ -8,5 +8,5 @@
   <xacro:property name="support_height" value="1.30" />
   <xacro:macro name="structure" params="parent child body_height body_width body_large">
-      <xacro:joint_pos_transmission joint="beam_to_slider"/>
+    <!--xacro:joint_pos_transmission joint="beam_to_slider"/-->
     <gazebo reference="support_to_base_link">
       <provideFeedback>true</provideFeedback>
@@ -22,5 +22,5 @@
     <origin xyz="0 0 0" rpy="0 0 0" />
   </joint>
-  <joint name="column_to_beam" type="fixed">
+  <joint name="column_to_beam" type="continuous">
     <parent link="column"/>
     <child link="beam"/>
@@ -28,10 +28,10 @@
     <origin xyz="0 0 ${column_height/2}" rpy="0 0 0" />
   </joint>
-    <joint name="slider_to_support" type="fixed">
+    <joint name="slider_to_support" type="prismatic">
     <parent link="slider"/>
     <child link="support"/>
     <origin xyz="0 0 ${-1*(cross_length/2)}" rpy="0 0 0" />
-    <axis xyz="0 1 0" />
-    <!--limit effort="15" velocity="50" lower="${-90*M_PI/180}" upper="${90*M_PI/180}" /-->
+    <axis xyz="0 0 1" />
+    <limit effort="15" velocity="50" lower="0" upper="1" />
   </joint>
   <joint name="support_to_base_link" type="fixed">
@@ -40,10 +40,10 @@
     <origin xyz="0 0 ${-support_height}" rpy="0 0 0" />
   </joint>
-  <joint name="beam_to_slider" type="prismatic">
+  <joint name="beam_to_slider" type="fixed">
     <parent link="beam"/>
     <child link="slider"/>
     <origin xyz="0 5 ${-1*cross_length}" rpy="0 0 0"/>
     <axis xyz="1 0 0" />
-    <limit effort="3" velocity="2" lower="5" upper="20" />
+    <!--limit effort="3" velocity="2" lower="5" upper="20" /-->
   </joint>
   <link name="column">
@@ -60,10 +60,10 @@
       </geometry>
     </visual>
-    <collision>
+    <!--collision>
       <origin xyz="0 0 0" rpy="0 0 0" />
       <geometry>
         <box size="${cross_length} ${cross_length} ${column_height}" />
       </geometry>
-    </collision>
+    </collision-->
   </link>
     <link name="slider">
@@ -79,13 +79,13 @@
       </geometry>
     </visual>
-    <collision>
+    <!--collision>
       <geometry>
         <box size="${cross_length} ${cross_length} ${cross_length}" />
       </geometry>
-    </collision>
+    </collision-->
   </link>
     <link name="support">
     <inertial>
-      <origin xyz="0 0 0" />
+      <origin xyz="0 0 ${-1*support_height/2}" />
       <mass value="0.4"/>
       <xacro:cuboid_inertia_def x="${cross_length}" y="${cross_length}" z="${support_height}" mass="0.4"/>
@@ -97,14 +97,14 @@
       </geometry>
     </visual>
-    <collision>
+    <!--collision>
       <origin xyz="0 0 ${-1*support_height/2}" rpy="0 0 0" />
       <geometry>
         <box size="${cross_length} ${cross_length} ${support_height}" />
       </geometry>
-    </collision>
+    </collision-->
   </link>
     <link name="beam">
     <inertial>
-      <origin xyz="0 ${beam_height/2} 0" />
+      <origin xyz="0 ${beam_height/2} 0" rpy="0 0 ${90*M_PI/180}"/>
       <mass value="8"/>
       <xacro:cuboid_inertia_def x="${cross_length}" y="${beam_height}" z="${cross_length}" mass="8"/>
@@ -117,10 +117,10 @@
       </geometry>
     </visual>
-    <collision>
+    <!--collision>
       <origin xyz="0 ${beam_height/2} 0" rpy="0 0 0" />
       <geometry>
         <box size="${cross_length} ${beam_height} ${cross_length} " />
       </geometry>
-    </collision>
+    </collision-->
   </link>
 </xacro:macro>

Commit message: ahora no colapsa

File: urdf/details.xacro (robot description, xacro)
@@ -19,6 +19,6 @@
     <inertial>
       <origin xyz="0 0 0" />
-      <mass value="0.01"/>
-      <xacro:cuboid_inertia_def x="${body_large/7}" y="${body_width/7}" z="${body_height/7}" mass="0.01"/>
+      <mass value="0.1"/>
+      <xacro:cuboid_inertia_def x="${body_large/7}" y="${body_width/7}" z="${body_height/7}" mass="0.1"/>
     </inertial>
     <visual>
@@ -40,6 +40,6 @@
     <inertial>
       <origin xyz="${body_large/4} 0 0" />
-      <mass value="0.5"/>
-      <xacro:cuboid_inertia_def x="${body_large/2}" y="${body_width*0.8}" z="${body_height*0.6}" mass="0.5"/>
+      <mass value="5"/>
+      <xacro:cuboid_inertia_def x="${body_large/2}" y="${body_width*0.8}" z="${body_height*0.6}" mass="5"/>
     </inertial>
     <visual>
@@ -61,6 +61,6 @@
     <inertial>
       <origin xyz="-0.200 0 0" />
-      <mass value="0.6"/>
-      <xacro:cuboid_inertia_def x="${body_large*2}" y="${body_width}" z="${body_height/2}" mass="0.6"/>
+      <mass value="6"/>
+      <xacro:cuboid_inertia_def x="${body_large*2}" y="${body_width}" z="${body_height/2}" mass="6"/>
     </inertial>
     <visual>

File: urdf/experiment.xacro (robot description, xacro)
@@ -18,6 +18,6 @@
     <inertial>
       <origin xyz="0 0 0" />
-      <mass value="0.8"/>
-      <xacro:cuboid_inertia_def x="${body_large}" y="${body_width}" z="${body_height}" mass="0.8"/>
+      <mass value="8"/>
+      <xacro:cuboid_inertia_def x="${body_large}" y="${body_width}" z="${body_height}" mass="8"/>
     </inertial>
     <visual>

File: urdf/leg.xacro (robot description, xacro)
@@ -31,7 +31,7 @@
   <xacro:macro name="cuboid_inertia_def" params="x y z mass">
     <inertia
-      iyy="${mass*(z*z+x*x)/12.0}"
-      ixx="${mass*(y*y+z*z)/12.0}"
-      izz="${mass*(x*x+y*y)/12.0}"
+      iyy="${100000*mass*(z*z+x*x)/12.0}"
+      ixx="${100000*mass*(y*y+z*z)/12.0}"
+      izz="${100000*mass*(x*x+y*y)/12.0}"
       ixy="0.0" iyz="0.0" ixz="0.0"/>
   </xacro:macro>
@@ -45,6 +45,6 @@
     <inertial>
       <origin xyz="0 0 ${-1*pelvis_height/2}" />
-      <mass value="0.3"/>
-      <xacro:cuboid_inertia_def x="${pelvis_large}" y="${pelvis_width}" z="${pelvis_height}" mass="0.3"/>
+      <mass value="3"/>
+      <xacro:cuboid_inertia_def x="${pelvis_large}" y="${pelvis_width}" z="${pelvis_height}" mass="3"/>
     </inertial>
     <visual>
@@ -64,6 +64,6 @@
     <inertial>
       <origin xyz="0 0 0" />
-      <mass value="0.1"/>
-      <xacro:cuboid_inertia_def x="${thigh_virtual_large}" y="${thigh_virtual_width}" z="${thigh_virtual_height}" mass="0.6"/>
+      <mass value="1"/>
+      <xacro:cuboid_inertia_def x="${thigh_virtual_large}" y="${thigh_virtual_width}" z="${thigh_virtual_height}" mass="6"/>
     </inertial>
     <visual>
@@ -82,6 +82,6 @@
     <inertial>
       <origin xyz="0 0 ${-1*thigh_height/2}" />
-      <mass value="0.8"/>
-      <xacro:cuboid_inertia_def x="${thigh_large}" y="${thigh_width}" z="${thigh_height}" mass="0.8"/>
+      <mass value="8"/>
+      <xacro:cuboid_inertia_def x="${thigh_large}" y="${thigh_width}" z="${thigh_height}" mass="8"/>
     </inertial>
     <visual>
@@ -101,6 +101,6 @@
     <inertial>
       <origin xyz="0 0 ${-1*tibia_height/2}" />
-      <mass value="0.6"/>
-      <xacro:cuboid_inertia_def x="${tibia_large}" y="${tibia_width}" z="${tibia_height}" mass="0.6"/>
+      <mass value="6"/>
+      <xacro:cuboid_inertia_def x="${tibia_large}" y="${tibia_width}" z="${tibia_height}" mass="6"/>
     </inertial>
     <visual>
@@ -120,6 +120,6 @@
     <inertial>
       <origin xyz="0 0 ${-1*ankle_height/2}" />
-      <mass value="0.3"/>
-      <xacro:cuboid_inertia_def x="${ankle_large}" y="${ankle_width}" z="${ankle_height}" mass="0.3"/>
+      <mass value="3"/>
+      <xacro:cuboid_inertia_def x="${ankle_large}" y="${ankle_width}" z="${ankle_height}" mass="3"/>
     </inertial>
     <visual>
@@ -145,6 +145,6 @@
     <inertial>
       <origin xyz="0 0 ${-1*phalange_height/2}" />
-      <mass value="0.1"/>
-      <xacro:cuboid_inertia_def x="${phalange_large}" y="${phalange_width}" z="${phalange_height}" mass="0.1"/>
+      <mass value="1"/>
+      <xacro:cuboid_inertia_def x="${phalange_large}" y="${phalange_width}" z="${phalange_height}" mass="1"/>
     </inertial>
     <visual>

File: urdf/structure.xacro (robot description, xacro)
@@ -22,9 +22,10 @@
     <origin xyz="0 0 0" rpy="0 0 0" />
   </joint>
-  <joint name="column_to_beam" type="continuous">
+  <joint name="column_to_beam" type="prismatic">
     <parent link="column"/>
     <child link="beam"/>
     <axis xyz="0 0 1"/>
     <origin xyz="0 0 ${column_height/2}" rpy="0 0 0" />
+    <limit effort="3" velocity="3" lower="1" upper="2" />
   </joint>
     <joint name="slider_to_support" type="fixed">
@@ -40,10 +41,10 @@
     <origin xyz="0 0 ${-support_height}" rpy="0 0 0" />
   </joint>
-  <joint name="beam_to_slider" type="fixed">
+  <joint name="beam_to_slider" type="prismatic">
     <parent link="beam"/>
     <child link="slider"/>
-    <origin xyz="0 5 ${-1*cross_length}" rpy="0 0 0"/>
+    <origin xyz="0 5 ${-1*cross_length}" rpy="0 0 ${90*M_PI/180}"/>
     <axis xyz="1 0 0" />
-    <!--limit effort="3" velocity="2" lower="5" upper="20" /-->
+    <limit effort="3" velocity="2" lower="5" upper="20" />
   </joint>
   <link name="column">
@@ -70,6 +71,6 @@
     <inertial>
       <origin xyz="0 0 0" />
-      <mass value="0.1"/>
-      <xacro:cuboid_inertia_def x="${cross_length}" y="${cross_length}" z="${cross_length}" mass="0.1"/>
+      <mass value="1"/>
+      <xacro:cuboid_inertia_def x="${cross_length}" y="${cross_length}" z="${cross_length}" mass="1"/>
     </inertial>
     <visual>
@@ -88,6 +89,6 @@
     <inertial>
       <origin xyz="0 0 ${-1*support_height/2}" />
-      <mass value="0.4"/>
-      <xacro:cuboid_inertia_def x="${cross_length}" y="${cross_length}" z="${support_height}" mass="0.4"/>
+      <mass value="4"/>
+      <xacro:cuboid_inertia_def x="${cross_length}" y="${cross_length}" z="${support_height}" mass="4"/>
     </inertial>
     <visual>
@@ -107,6 +108,6 @@
     <inertial>
       <origin xyz="0 ${beam_height/2} 0" rpy="0 0 0"/>
-      <mass value="8"/>
-      <xacro:cuboid_inertia_def x="${cross_length}" y="${beam_height}" z="${cross_length}" mass="8"/>
+      <mass value="80"/>
+      <xacro:cuboid_inertia_def x="${cross_length}" y="${beam_height}" z="${cross_length}" mass="80"/>
     </inertial>
     <visual>

Commit message: maomeno

File: urdf/details.xacro (robot description, xacro)
@@ -61,6 +61,6 @@
     <inertial>
       <origin xyz="-0.200 0 0" />
-      <mass value="0.6"/>
-      <xacro:cuboid_inertia_def x="${body_large*2}" y="${body_width}" z="${body_height/2}" mass="0.6"/>
+      <mass value="0.5"/>
+      <xacro:cuboid_inertia_def x="${body_large*2}" y="${body_width}" z="${body_height/2}" mass="0.5"/>
     </inertial>
     <visual>

File: urdf/experiment.xacro (robot description, xacro)
@@ -18,6 +18,6 @@
     <inertial>
       <origin xyz="0 0 0" />
-      <mass value="0.8"/>
-      <xacro:cuboid_inertia_def x="${body_large}" y="${body_width}" z="${body_height}" mass="0.8"/>
+      <mass value="0.6"/>
+      <xacro:cuboid_inertia_def x="${body_large}" y="${body_width}" z="${body_height}" mass="0.6"/>
     </inertial>
     <visual>

File: urdf/leg.xacro (robot description, xacro)
@@ -45,6 +45,6 @@
     <inertial>
       <origin xyz="0 0 ${-1*pelvis_height/2}" />
-      <mass value="0.3"/>
-      <xacro:cuboid_inertia_def x="${pelvis_large}" y="${pelvis_width}" z="${pelvis_height}" mass="0.3"/>
+      <mass value="0.2"/>
+      <xacro:cuboid_inertia_def x="${pelvis_large}" y="${pelvis_width}" z="${pelvis_height}" mass="0.2"/>
     </inertial>
     <visual>
@@ -64,6 +64,6 @@
     <inertial>
       <origin xyz="0 0 0" />
-      <mass value="0.1"/>
-      <xacro:cuboid_inertia_def x="${thigh_virtual_large}" y="${thigh_virtual_width}" z="${thigh_virtual_height}" mass="0.6"/>
+      <mass value="0.05"/>
+      <xacro:cuboid_inertia_def x="${thigh_virtual_large}" y="${thigh_virtual_width}" z="${thigh_virtual_height}" mass="0.05"/>
     </inertial>
     <visual>
@@ -82,6 +82,6 @@
     <inertial>
       <origin xyz="0 0 ${-1*thigh_height/2}" />
-      <mass value="0.8"/>
-      <xacro:cuboid_inertia_def x="${thigh_large}" y="${thigh_width}" z="${thigh_height}" mass="0.8"/>
+      <mass value="0.25"/>
+      <xacro:cuboid_inertia_def x="${thigh_large}" y="${thigh_width}" z="${thigh_height}" mass="0.5"/>
     </inertial>
     <visual>
@@ -101,6 +101,6 @@
     <inertial>
       <origin xyz="0 0 ${-1*tibia_height/2}" />
-      <mass value="0.6"/>
-      <xacro:cuboid_inertia_def x="${tibia_large}" y="${tibia_width}" z="${tibia_height}" mass="0.6"/>
+      <mass value="0.2"/>
+      <xacro:cuboid_inertia_def x="${tibia_large}" y="${tibia_width}" z="${tibia_height}" mass="0.4"/>
     </inertial>
     <visual>
@@ -120,6 +120,6 @@
     <inertial>
       <origin xyz="0 0 ${-1*ankle_height/2}" />
-      <mass value="0.3"/>
-      <xacro:cuboid_inertia_def x="${ankle_large}" y="${ankle_width}" z="${ankle_height}" mass="0.3"/>
+      <mass value="0.2"/>
+      <xacro:cuboid_inertia_def x="${ankle_large}" y="${ankle_width}" z="${ankle_height}" mass="0.2"/>
     </inertial>
     <visual>
@@ -145,6 +145,6 @@
     <inertial>
       <origin xyz="0 0 ${-1*phalange_height/2}" />
-      <mass value="0.1"/>
-      <xacro:cuboid_inertia_def x="${phalange_large}" y="${phalange_width}" z="${phalange_height}" mass="0.1"/>
+      <mass value="0.07"/>
+      <xacro:cuboid_inertia_def x="${phalange_large}" y="${phalange_width}" z="${phalange_height}" mass="0.07"/>
     </inertial>
     <visual>

File: urdf/structure.xacro (robot description, xacro)
@@ -5,5 +5,5 @@
   <xacro:property name="column_height" value="1.25" />
   <xacro:property name="cross_length" value="0.025" />
-  <xacro:property name="beam_height" value="7" />
+  <xacro:property name="beam_height" value="10" />
   <xacro:property name="support_height" value="1.26" />
   <xacro:macro name="structure" params="parent child body_height body_width body_large">
@@ -43,5 +43,5 @@
     <parent link="beam"/>
     <child link="slider"/>
-    <origin xyz="0 5 ${-1*cross_length}" rpy="0 0 0"/>
+    <origin xyz="0 1 ${-1*cross_length}" rpy="0 0 0"/>
     <axis xyz="1 0 0" />
     <!--limit effort="3" velocity="2" lower="5" upper="20" /-->
@@ -51,5 +51,5 @@
       <origin xyz="0 0 0" />
       <mass value="3"/>
-      <xacro:cuboid_inertia_def x="${cross_length}" y="${cross_length}" z="${column_height}" mass="3"/>
+      <xacro:cuboid_inertia_def x="${cross_length}" y="${cross_length}" z="${column_height}" mass="30"/>
     </inertial>
     <visual>
@@ -60,10 +60,10 @@
       </geometry>
     </visual>
-    <!--collision>
+    <collision>
       <origin xyz="0 0 0" rpy="0 0 0" />
       <geometry>
         <box size="${cross_length} ${cross_length} ${column_height}" />
       </geometry>
-    </collision-->
+    </collision>
   </link>
     <link name="slider">
@@ -71,5 +71,5 @@
       <origin xyz="0 0 0" />
       <mass value="0.1"/>
-      <xacro:cuboid_inertia_def x="${cross_length}" y="${cross_length}" z="${cross_length}" mass="0.1"/>
+      <xacro:cuboid_inertia_def x="${cross_length}" y="${cross_length}" z="${cross_length}" mass="1"/>
     </inertial>
     <visual>
@@ -79,9 +79,9 @@
       </geometry>
     </visual>
-    <!--collision>
+    <collision>
       <geometry>
         <box size="${cross_length} ${cross_length} ${cross_length}" />
       </geometry>
-    </collision-->
+    </collision>
   </link>
     <link name="support">
@@ -89,5 +89,5 @@
       <origin xyz="0 0 ${-1*support_height/2}" />
       <mass value="0.4"/>
-      <xacro:cuboid_inertia_def x="${cross_length}" y="${cross_length}" z="${support_height}" mass="0.4"/>
+      <xacro:cuboid_inertia_def x="${cross_length}" y="${cross_length}" z="${support_height}" mass="4"/>
     </inertial>
     <visual>
@@ -97,10 +97,10 @@
       </geometry>
     </visual>
-    <!--collision>
+    <collision>
       <origin xyz="0 0 ${-1*support_height/2}" rpy="0 0 0" />
       <geometry>
         <box size="${cross_length} ${cross_length} ${support_height}" />
       </geometry>
-    </collision-->
+    </collision>
   </link>
     <link name="beam">
@@ -108,5 +108,5 @@
       <origin xyz="0 ${beam_height/2} 0" rpy="0 0 0"/>
       <mass value="8"/>
-      <xacro:cuboid_inertia_def x="${cross_length}" y="${beam_height}" z="${cross_length}" mass="8"/>
+      <xacro:cuboid_inertia_def x="${cross_length}" y="${beam_height}" z="${cross_length}" mass="80"/>
     </inertial>
     <visual>
@@ -117,10 +117,10 @@
       </geometry>
     </visual>
-    <!--collision>
+    <collision>
       <origin xyz="0 ${beam_height/2} 0" rpy="0 0 0" />
       <geometry>
         <box size="${cross_length} ${beam_height} ${cross_length} " />
       </geometry>
-    </collision-->
+    </collision>
   </link>
 </xacro:macro>

Commit message: no camina pero gatea

File: urdf/details.xacro (robot description, xacro)
@@ -40,6 +40,6 @@
     <inertial>
       <origin xyz="${body_large/4} 0 0" />
-      <mass value="0.5"/>
-      <xacro:cuboid_inertia_def x="${body_large/2}" y="${body_width*0.8}" z="${body_height*0.6}" mass="0.5"/>
+      <mass value="0.8"/>
+      <xacro:cuboid_inertia_def x="${body_large/2}" y="${body_width*0.8}" z="${body_height*0.6}" mass="0.8"/>
     </inertial>
     <visual>

File: urdf/experiment.xacro (robot description, xacro)
@@ -18,6 +18,6 @@
     <inertial>
       <origin xyz="0 0 0" />
-      <mass value="0.8"/>
-      <xacro:cuboid_inertia_def x="${body_large}" y="${body_width}" z="${body_height}" mass="0.8"/>
+      <mass value="1.5"/>
+      <xacro:cuboid_inertia_def x="${body_large}" y="${body_width}" z="${body_height}" mass="1.5"/>
     </inertial>
     <visual>

File: urdf/structure.xacro (robot description, xacro)
@@ -19,9 +19,10 @@
     <origin xyz="0 0 ${-column_height/2}" rpy="0 0 0" />
   </joint>
-  <joint name="beam_to_base_link" type="fixed">
+  <joint name="beam_to_base_link" type="revolute">
     <parent link="beam"/>
     <child link="${child}"/>
     <origin xyz="0 ${beam_height} 0" rpy="0 0 0" />
-    <!--limit effort="4" velocity="4" lower="0" upper="0.01" /-->
+      <axis xyz="0 1 0"/>
+    <limit effort="4" velocity="4" lower="-1" upper="1" />
   </joint>
   <link name="column">

Commit message: camina

File: urdf/details.xacro (robot description, xacro)
@@ -4,16 +4,16 @@
   name="details">
   <xacro:macro name="details" params="parent body_height body_width body_large">
- <gazebo reference="body_to_tail">
+ <!--gazebo reference="body_to_tail">
       <provideFeedback>true</provideFeedback>
       <disableFixedJointLumping>true</disableFixedJointLumping>
-    </gazebo>
+    </gazebo-->
    <!--gazebo reference="neck_to_head">
       <provideFeedback>true</provideFeedback>
       <disableFixedJointLumping>true</disableFixedJointLumping>
     </gazebo-->
-    <gazebo reference="body_to_neck">
+    <!--gazebo reference="body_to_neck">
       <provideFeedback>true</provideFeedback>
       <disableFixedJointLumping>true</disableFixedJointLumping>
-    </gazebo>
+    </gazebo-->
  <link name="neck">
     <inertial>
@@ -40,6 +40,6 @@
     <inertial>
       <origin xyz="${body_large/4} 0 0" />
-      <mass value="0.8"/>
-      <xacro:cuboid_inertia_def x="${body_large/2}" y="${body_width*0.8}" z="${body_height*0.6}" mass="0.8"/>
+      <mass value="1.5"/>
+      <xacro:cuboid_inertia_def x="${body_large/2}" y="${body_width*0.8}" z="${body_height*0.6}" mass="1.5"/>
     </inertial>
     <visual>

File: urdf/experiment.xacro (robot description, xacro)
@@ -18,6 +18,6 @@
     <inertial>
       <origin xyz="0 0 0" />
-      <mass value="1.5"/>
-      <xacro:cuboid_inertia_def x="${body_large}" y="${body_width}" z="${body_height}" mass="1.5"/>
+      <mass value="1.7"/>
+      <xacro:cuboid_inertia_def x="${body_large}" y="${body_width}" z="${body_height}" mass="1.7"/>
     </inertial>
     <visual>

Commit message: final commit

File: urdf/details.xacro (robot description, xacro)
@@ -40,6 +40,6 @@
     <inertial>
       <origin xyz="${body_large/4} 0 0" />
-      <mass value="1.5"/>
-      <xacro:cuboid_inertia_def x="${body_large/2}" y="${body_width*0.8}" z="${body_height*0.6}" mass="1.5"/>
+      <mass value="1"/>
+      <xacro:cuboid_inertia_def x="${body_large/2}" y="${body_width*0.8}" z="${body_height*0.6}" mass="1"/>
     </inertial>
     <visual>
@@ -61,6 +61,6 @@
     <inertial>
       <origin xyz="-0.200 0 0" />
-      <mass value="0.5"/>
-      <xacro:cuboid_inertia_def x="${body_large*2}" y="${body_width}" z="${body_height/2}" mass="0.5"/>
+      <mass value="0.4"/>
+      <xacro:cuboid_inertia_def x="${body_large*2}" y="${body_width}" z="${body_height/2}" mass="0.4"/>
     </inertial>
     <visual>

File: urdf/experiment.xacro (robot description, xacro)
@@ -18,6 +18,6 @@
     <inertial>
       <origin xyz="0 0 0" />
-      <mass value="1.7"/>
-      <xacro:cuboid_inertia_def x="${body_large}" y="${body_width}" z="${body_height}" mass="1.7"/>
+      <mass value="1.0"/>
+      <xacro:cuboid_inertia_def x="${body_large}" y="${body_width}" z="${body_height}" mass="1.0"/>
     </inertial>
     <visual>

File: urdf/leg.xacro (robot description, xacro)
@@ -120,6 +120,6 @@
     <inertial>
       <origin xyz="0 0 ${-1*ankle_height/2}" />
-      <mass value="0.05"/>
-      <xacro:cuboid_inertia_def x="${ankle_large}" y="${ankle_width}" z="${ankle_height}" mass="0.05"/>
+      <mass value="0.2"/>
+      <xacro:cuboid_inertia_def x="${ankle_large}" y="${ankle_width}" z="${ankle_height}" mass="0.2"/>
     </inertial>
     <visual>
@@ -145,6 +145,6 @@
     <inertial>
       <origin xyz="0 0 ${-1*phalange_height/2}" />
-      <mass value="0.06"/>
-      <xacro:cuboid_inertia_def x="${phalange_large}" y="${phalange_width}" z="${phalange_height}" mass="0.06"/>
+      <mass value="0.2"/>
+      <xacro:cuboid_inertia_def x="${phalange_large}" y="${phalange_width}" z="${phalange_height}" mass="0.2"/>
     </inertial>
     <visual>
